File: hdw/LED board/LED Board/POS3P3_Supply.kicad_sch (KiCad schematic)
At the start: 0 parts

Commit message: started POS3P3 supply. Need to finish choosing discretes, especially sense resistors on both LED supply and 3p3 supply
Parts:
- added C401, C406: 0.1uF, Capacitors_SMD:C_0402, symbol Custom_Library:C_Custom
- added C402, C404: 10uF, Capacitors_SMD:C_1206, symbol Custom_Library:C_Custom
- added C403, C407, C408: 10uF, Capacitors_SMD:C_0805, symbol Custom Library:C_Custom
- added C405: 10nF, Capacitors_SMD:C_0402, symbol Custom_Library:C_Custom
- added D401: BAT48JFILM, Diode_SMD:D_SOD-323, symbol Diode:BAT48JFILM
- added L401: 2.2uH, Inductors_SMD:L_Vishay_IHLP-2020, symbol Custom_Library:L_Custom
- added Q401: BSS214NW, Package_TO_SOT_SMD:SOT-323_SC-70, symbol Transistor_FET:BSS214NW
- added Q402: ZXMS6004FFTA, Package_TO_SOT_SMD:SOT-23, symbol Custom_Library:ZXMS6004FFTA
- added R401, R406: 0, Resistors_SMD:R_0402, symbol Custom_Library:R_Custom
- added R402, R403, R404: 10k, Resistors_SMD:R_0402, symbol Custom_Library:R_Custom
- added R405, R408: 10, Resistors_SMD:R_0402, symbol Custom_Library:R_Custom
- added R407: 0.02, Resistors_SMD:R_0612, symbol Custom_Library:R_Custom
- added R409: 3.16k, Resistors_SMD:R_0402, symbol Custom_Library:R_Custom
- added R410: 1k, Resistors_SMD:R_0402, symbol Custom_Library:R_Custom
- added TP401: TP, Custom Footprints Library:Test_Point, symbol Custom_Library:TP
- added U401: 74LVC1G97, Package_TO_SOT_SMD:SOT-363_SC-70-6, symbol Custom_Library:74LVC1G97_Power_AND
- added U402: TPS62130A, Package_DFN_QFN:QFN-16-1EP_3x3mm_P0.5mm_EP1.75x1.75mm, symbol Custom_Library:TPS62130
Connections:
- new net: C403.1, D401.1 (K), R404.1
- new net: R403.2, U401.6, U402.4 (PG)
- new net: R406.1, R409.2, R410.1, U402.5 (FB)
- new net: L401.1, U402.1 (SW), U402.2 (SW), U402.3 (SW)
- new net: C405.1, U402.9 (SS/TR)
- new net: C407.1, C408.1, L401.2, R405.2, R407.1
- new net: Q401.3 (D), Q402.1 (G), R404.2
- new net +12V: C402.1, C404.1, C406.1, U402.10 (AVIN), U402.11 (PVIN), U402.12 (PVIN)
- new net +3.3V: C401.1, D401.2 (A), Q402.3 (D), R403.1, R407.2, R408.2, R409.1, TP401.1 (TP), U401.5 (VCC), U402.14 (VOS)
- new net GND: C401.2, C402.2, C403.2, C404.2, C405.2, C406.2, C407.2, C408.2, Q401.2 (S), Q402.2 (S), R402.2, R406.2, R410.2, U401.1 (GND), U401.2 (GND), U402.15 (PGND), U402.16 (PGND), U402.17 (EP), U402.6 (AGND), U402.7 (FSW), U402.8 (DEF)
- new net POS12_PGOOD: R401.1
- new net POS3P3_PGOOD: R402.1, U401.4
- new net POS3P3_RUN: Q401.1 (G), R401.2, U401.3, U402.13 (EN)
- new net POS3P3_SNS+: R405.1
- new net POS3P3_SNS-: R408.1
Other:
- note added: "TRY TO TALLY LOAD CURRENTS"

Commit message: forgot to push pdf
Parts:
- removed C404: 10uF, Capacitors_SMD:C_1206, symbol Custom_Library:C_Custom
- removed C407, C408: 10uF, Capacitors_SMD:C_0805, symbol Custom Library:C_Custom
- added C? (x2): 10uF, Capacitors_SMD:C_1206, symbol Custom_Library:C_Custom
- L401: footprint Inductors_SMD:L_Vishay_IHLP-2020 -> Inductor_SMD:L_Vishay_IHLP-2020; Ampacity 6.7A -> 5.8A; Digi-Key PN 541-1236-1-ND -> (none)
- U402: value TPS62130A -> TPS62150A; Digi-Key PN 296-39446-1-ND -> (none)
Connections:
- net GND: now also C?.2, C?.2
- net at L401.2, R405.2, R407.1: now also C?.1, C?.1
Other:
- moved on the sheet: C402
