File: hdw/LED board/LED Board/LED_Driver_15.kicad_sch (KiCad schematic)
At the start: 21 parts

Commit message: added connectors, updated some signal names on labels
Parts:
- removed C?: 0.1uF, symbol Custom Library:C_Custom
- removed D? (x10): GREEN, symbol Device:LED
- removed D? (x2): RED, symbol Device:LED
- removed D?: YELLOW, symbol Device:LED
- removed R?: 2.52k, Resistor_THT:R_Array_SIP4, symbol Custom Library:R_Custom
- removed R?: 10k, symbol Custom Library:R_Custom
- removed U?: TLC59281RGER, TLC59281RGER:QFN50P400X400X100-25N, symbol TLC59281RGER:TLC59281RGER
- added C?: 0.1uF, symbol Custom Library:C_Custom
- added D? (x10): GREEN, symbol Device:LED
- added D?: YELLOW, symbol Device:LED
- added D? (x2): RED, symbol Device:LED
- added R?: 2.52k, Resistor_THT:R_Array_SIP4, symbol Custom Library:R_Custom
- added R?: 10k, symbol Custom Library:R_Custom
- added U?: TLC59281RGER, TLC59281RGER:QFN50P400X400X100-25N, symbol TLC59281RGER:TLC59281RGER
Connections:
- net +3.3V: now also C?.1, U?.21 (VCC)
- net BLANK: now also U?.18 (BLANK)
- net GND: now also C?.2, R?.2, R?.2, U?.22 (GND), U?.25 (EP)
- net LAT: now also U?.1 (LAT)
- net SCLK: now also U?.24 (SCLK)
- net SIN_15: now also R?.1, U?.23 (SIN)
- net VLED: now also D?.2 (A), D?.2 (A), D?.2 (A), D?.2 (A), D?.2 (A), D?.2 (A), D?.2 (A), D?.2 (A), D?.2 (A), D?.2 (A), D?.2 (A), D?.2 (A), D?.2 (A)
- net at R?.1: now also U?.19 (SOUT)
- net at D11.1 (K): now also U?.12 (OUT10)
- net at D12.1 (K): now also U?.13 (OUT11)
- net at D13.1 (K): now also U?.14 (OUT12)
- new net: D?.1 (K), U?.2 (OUT0)
- new net: D?.1 (K), U?.7 (OUT5)
- new net: D?.1 (K), U?.4 (OUT2)
- new net: D?.1 (K), U?.3 (OUT1)
- new net: D?.1 (K), U?.6 (OUT4)
- new net: D?.1 (K), U?.11 (OUT9)
- new net: R?.1, U?.20 (IREF)
- new net: D?.1 (K), U?.8 (OUT6)
- new net: D?.1 (K), U?.10 (OUT8)
- new net: D?.1 (K), U?.15 (OUT13)
- new net: D?.1 (K), U?.16 (OUT14)
- new net: D?.1 (K), U?.17 (OUT15)
- new net: D?.1 (K), U?.5 (OUT3)
- new net: D?.1 (K), U?.9 (OUT7)
