File: hdw/LED board/LED Board/led_panel_connector.kicad_sch (KiCad schematic)
At the start: 4 parts, among them J20001 Left

Commit message: fixed footprint issue on protection circuit
Parts:
- D20001, D20002: footprint project_lib:SOT-323_SC-70 -> project_lib:SOT-363_SC-70-6
Changed lines of the file:
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@@
 			)
 		)
-		(property "Footprint" "project_lib:SOT-323_SC-70"
+		(property "Footprint" "project_lib:SOT-363_SC-70-6"
 			(at 60.96 66.04 0)
 			(hide yes)
@@
 			)
 		)
-		(property "Footprint" "project_lib:SOT-323_SC-70"
+		(property "Footprint" "project_lib:SOT-363_SC-70-6"
 			(at 99.06 66.04 0)
 			(hide yes)
@@
 			)
 		)
-		(property "Footprint" "project_lib:SOT-323_SC-70"
+		(property "Footprint" "project_lib:SOT-363_SC-70-6"
 			(at 41.91 66.04 0)
 			(hide yes)
@@
 			)
 		)
-		(property "Footprint" "project_lib:SOT-323_SC-70"
+		(property "Footprint" "project_lib:SOT-363_SC-70-6"
 			(at 67.31 66.04 0)
 			(hide yes)
@@
 			)
 		)
-		(property "Footprint" "project_lib:SOT-323_SC-70"
+		(property "Footprint" "project_lib:SOT-363_SC-70-6"
 			(at 54.61 66.04 0)
 			(hide yes)
@@
 			)
 		)
-		(property "Footprint" "project_lib:SOT-323_SC-70"
+		(property "Footprint" "project_lib:SOT-363_SC-70-6"
 			(at 118.11 66.04 0)
 			(hide yes)
@@
 			)
 		)
-		(property "Footprint" "project_lib:SOT-323_SC-70"
+		(property "Footprint" "project_lib:SOT-363_SC-70-6"
 			(at 92.71 66.04 0)
 			(hide yes)
@@
 			)
 		)
-		(property "Footprint" "project_lib:SOT-323_SC-70"
+		(property "Footprint" "project_lib:SOT-363_SC-70-6"
 			(at 105.41 66.04 0)
 			(hide yes)
@@
 			)
 		)
-		(property "Footprint" "project_lib:SOT-323_SC-70"
+		(property "Footprint" "project_lib:SOT-363_SC-70-6"
 			(at 111.76 66.04 0)
 			(hide yes)
@@
 			)
 		)
-		(property "Footprint" "project_lib:SOT-323_SC-70"
+		(property "Footprint" "project_lib:SOT-363_SC-70-6"
 			(at 48.26 66.04 0)
 			(hide yes)
