File: hdw/DSP_board/rev_a/Audio_Visualiser_DSP/filtering_pgas.kicad_sch (KiCad schematic)
At the start: 28 parts

Commit message: Added a ton of shit. I2C digipots, adjustable gain op amps, broke out audio references
Parts:
- added U? (x2): MCP4451-xxxx-ST, Package_SO:TSSOP-20_4.4x6.5mm_P0.65mm, symbol Potentiometer_Digital:MCP4451-xxxx-ST
Connections:
- net at R?.2: now also U?.12 (P0W); no longer U?.3
- net at R?.2: no longer U?.9
- new net: U?.11 (P0A), U?.3
Other:
- note added: "Verify rail to rail"
- moved on the sheet: C?, R?, U?A, U?B, U?C, U?D, U?E
