File: hdw/DSP_board/rev_a/Audio_Visualiser_DSP/anti_alias_filtering.kicad_sch (KiCad schematic)
At the start: 23 parts

Commit message: Added some spice models
Parts:
- gave numbers to parts that had none: 19

Commit message: added simulation, changed LPF VCC to +5V
Connections:
- net +3.3V renamed +5V

Commit message: more signal chain development and simulation
Parts:
- renumbered R71 to R73, R72 to R74, R73 to R75, R74 to R76, R75 to R77, R76 to R78, R77 to R79, R78 to R80
Other:
- note added: "Move to MCP6024"
- note removed: "Verify rail to rail"
- note removed: "Verify this will work with DC offset"
Changed lines of the file:
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@@
 		(date "2023-12-25")
 	)
-	(text "Verify this will work\nwith DC offset"
+	(text "Move to MCP6024"
 		(exclude_from_sim no)
-		(at 142.24 81.28 0)
+		(at 140.97 96.52 0)
 		(effects
 			(font
@@
 		)
 	)
-	(text "Verify rail to rail"
-		(exclude_from_sim no)
-		(at 142.24 106.68 0)
-		(effects
-			(font
-				(size 3.81 3.81)
-				(thickness 0.762)
-				(bold yes)
-				(color 194 0 0 1)
-			)
-		)
-	)
 	(junction
 		(at 147.32 114.3)
@@
 		(in_pos_files yes)
 		(dnp no)
-		(property "Reference" "#PWR0262"
+		(property "Reference" "#PWR0271"
 			(at 137.16 34.29 0)
 			(hide yes)
@@
 			(project "Audio_Visualiser_DSP"
 				(path "/97a4dfb8-0e16-46f1-9709-8d2007dd0cd3/f2b9a82c-2733-4630-b590-b588e09b6263"
-					(reference "#PWR0262")
+					(reference "#PWR0271")
 					(unit 1)
 				)
@@
 		(in_pos_files yes)
 		(dnp no)
-		(property "Reference" "#PWR0260"
+		(property "Reference" "#PWR0269"
 			(at 119.38 62.23 0)
 			(hide yes)
@@
 			(project "Audio_Visualiser_DSP"
 				(path "/97a4dfb8-0e16-46f1-9709-8d2007dd0cd3/f2b9a82c-2733-4630-b590-b588e09b6263"
-					(reference "#PWR0260")
+					(reference "#PWR0269")
 					(unit 1)
 				)
@@
 		(in_pos_files yes)
 		(dnp no)
-		(property "Reference" "#PWR0264"
+		(property "Reference" "#PWR0273"
 			(at 154.94 34.29 0)
 			(hide yes)
@@
 			(project "Audio_Visualiser_DSP"
 				(path "/97a4dfb8-0e16-46f1-9709-8d2007dd0cd3/f2b9a82c-2733-4630-b590-b588e09b6263"
-					(reference "#PWR0264")
+					(reference "#PWR0273")
 					(unit 1)
 				)
@@
 		(in_pos_files yes)
 		(dnp no)
-		(property "Reference" "R77"
+		(property "Reference" "R79"
 			(at 153.67 60.96 90)
 			(show_name no)
@@
 			(project "Audio_Visualiser_DSP"
 				(path "/97a4dfb8-0e16-46f1-9709-8d2007dd0cd3/f2b9a82c-2733-4630-b590-b588e09b6263"
-					(reference "R77")
+					(reference "R79")
 					(unit 1)
 				)
@@
 		(in_pos_files yes)
 		(dnp no)
-		(property "Reference" "#PWR0258"
+		(property "Reference" "#PWR0267"
 			(at 101.6 82.55 0)
 			(hide yes)
@@
 			(project "Audio_Visualiser_DSP"
 				(path "/97a4dfb8-0e16-46f1-9709-8d2007dd0cd3/f2b9a82c-2733-4630-b590-b588e09b6263"
-					(reference "#PWR0258")
+					(reference "#PWR0267")
 					(unit 1)
 				)
@@
 		(in_pos_files yes)
 		(dnp no)
-		(property "Reference" "#PWR0259"
+		(property "Reference" "#PWR0268"
 			(at 101.6 133.35 0)
 			(hide yes)
@@
 			(project "Audio_Visualiser_DSP"
 				(path "/97a4dfb8-0e16-46f1-9709-8d2007dd0cd3/f2b9a82c-2733-4630-b590-b588e09b6263"
-					(reference "#PWR0259")
+					(reference "#PWR0268")
 					(unit 1)
 				)
@@
 		(in_pos_files yes)
 		(dnp no)
-		(property "Reference" "R73"
+		(property "Reference" "R75"
 			(at 91.44 60.96 90)
 			(show_name no)
@@
 			(project "Audio_Visualiser_DSP"
 				(path "/97a4dfb8-0e16-46f1-9709-8d2007dd0cd3/f2b9a82c-2733-4630-b590-b588e09b6263"
-					(reference "R73")
+					(reference "R75")
 					(unit 1)
 				)
@@
 		(in_pos_files yes)
 		(dnp no)
-		(property "Reference" "#PWR0261"
+		(property "Reference" "#PWR0270"
 			(at 119.38 80.01 0)
 			(hide yes)
@@
 			(project "Audio_Visualiser_DSP"
 				(path "/97a4dfb8-0e16-46f1-9709-8d2007dd0cd3/f2b9a82c-2733-4630-b590-b588e09b6263"
-					(reference "#PWR0261")
+					(reference "#PWR0270")
 					(unit 1)
 				)
@@
 		(in_pos_files yes)
 		(dnp no)
-		(property "Reference" "#PWR0263"
+		(property "Reference" "#PWR0272"
 			(at 137.16 44.45 0)
 			(hide yes)
@@
 			(project "Audio_Visualiser_DSP"
 				(path "/97a4dfb8-0e16-46f1-9709-8d2007dd0cd3/f2b9a82c-2733-4630-b590-b588e09b6263"
-					(reference "#PWR0263")
+					(reference "#PWR0272")
 					(unit 1)
 				)
@@
 		(in_pos_files yes)
 		(dnp no)
-		(property "Reference" "R71"
+		(property "Reference" "R73"
 			(at 78.74 60.96 90)
 			(show_name no)
@@
 			(project "Audio_Visualiser_DSP"
 				(path "/97a4dfb8-0e16-46f1-9709-8d2007dd0cd3/f2b9a82c-2733-4630-b590-b588e09b6263"
-					(reference "R71")
+					(reference "R73")
 					(unit 1)
 				)
@@
 		(in_pos_files yes)
 		(dnp no)
-		(property "Reference" "#PWR0267"
+		(property "Reference" "#PWR0276"
 			(at 163.83 133.35 0)
 			(hide yes)
@@
 			(project "Audio_Visualiser_DSP"
 				(path "/97a4dfb8-0e16-46f1-9709-8d2007dd0cd3/f2b9a82c-2733-4630-b590-b588e09b6263"
-					(reference "#PWR0267")
+					(reference "#PWR0276")
 					(unit 1)
 				)
@@
 		(in_pos_files yes)
 		(dnp no)
-		(property "Reference" "R72"
+		(property "Reference" "R74"
 			(at 78.74 111.76 90)
 			(show_name no)
@@
 			(project "Audio_Visualiser_DSP"
 				(path "/97a4dfb8-0e16-46f1-9709-8d2007dd0cd3/f2b9a82c-2733-4630-b590-b588e09b6263"
-					(reference "R72")
+					(reference "R74")
 					(unit 1)
 				)
@@
 		(in_pos_files yes)
 		(dnp no)
-		(property "Reference" "R75"
+		(property "Reference" "R77"
 			(at 140.97 60.96 90)
 			(show_name no)
@@
 			(project "Audio_Visualiser_DSP"
 				(path "/97a4dfb8-0e16-46f1-9709-8d2007dd0cd3/f2b9a82c-2733-4630-b590-b588e09b6263"
-					(reference "R75")
+					(reference "R77")
 					(unit 1)
 				)
@@
 		(in_pos_files yes)
 		(dnp no)
-		(property "Reference" "R76"
+		(property "Reference" "R78"
 			(at 140.97 111.76 90)
 			(show_name no)
@@
 			(project "Audio_Visualiser_DSP"
 				(path "/97a4dfb8-0e16-46f1-9709-8d2007dd0cd3/f2b9a82c-2733-4630-b590-b588e09b6263"
-					(reference "R76")
+					(reference "R78")
 					(unit 1)
 				)
@@
 		(in_pos_files yes)
 		(dnp no)
-		(property "Reference" "R78"
+		(property "Reference" "R80"
 			(at 153.67 111.76 90)
 			(show_name no)
@@
 			(project "Audio_Visualiser_DSP"
 				(path "/97a4dfb8-0e16-46f1-9709-8d2007dd0cd3/f2b9a82c-2733-4630-b590-b588e09b6263"
-					(reference "R78")
+					(reference "R80")
 					(unit 1)
 				)
@@
 		(in_pos_files yes)
 		(dnp no)
-		(property "Reference" "R74"
+		(property "Reference" "R76"
 			(at 91.44 111.76 90)
 			(show_name no)
@@
 			(project "Audio_Visualiser_DSP"
 				(path "/97a4dfb8-0e16-46f1-9709-8d2007dd0cd3/f2b9a82c-2733-4630-b590-b588e09b6263"
-					(reference "R74")
+					(reference "R76")
 					(unit 1)
 				)
@@
 		(in_pos_files yes)
 		(dnp no)
-		(property "Reference" "#PWR0266"
+		(property "Reference" "#PWR0275"
 			(at 163.83 82.55 0)
 			(hide yes)
@@
 			(project "Audio_Visualiser_DSP"
 				(path "/97a4dfb8-0e16-46f1-9709-8d2007dd0cd3/f2b9a82c-2733-4630-b590-b588e09b6263"
-					(reference "#PWR0266")
+					(reference "#PWR0275")
 					(unit 1)
 				)
@@
 		(in_pos_files yes)
 		(dnp no)
-		(property "Reference" "#PWR0265"
+		(property "Reference" "#PWR0274"
 			(at 154.94 44.45 0)
 			(hide yes)
@@
 			(project "Audio_Visualiser_DSP"
 				(path "/97a4dfb8-0e16-46f1-9709-8d2007dd0cd3/f2b9a82c-2733-4630-b590-b588e09b6263"
-					(reference "#PWR0265")
+					(reference "#PWR0274")
 					(unit 1)
 				)

Commit message: changed to MCP6024 op amps for rail to rail inputs. Further simulated signal chain
Parts:
- U26: value MCP604 -> MCP6024
Connections:
- net +5V renamed +3.3V
Other:
- note removed: "10pF to GND?"
- note removed: "Move to MCP6024"

Commit message: added rotary encoder circuitry
Other:
- note added: "4-pole Sallen-Key active anti-aliasing lowpass filters Unity gain fc = 23.2kHz, Q = 0.707 each If sampling at 44.1kHz, nyquist is 22.05kHz Must filter hard around this frequency"
- note removed: "4-pole Sallen-Key active anti-aliasing lowpass filters Unity gain fc = 23.2kHz, Q = 0.707 each If sampling at 44.1kHz, nyquist is 22.05kHz Must filter hard just below this"
Changed lines of the file:
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@@
 		(date "2023-12-25")
 	)
-	(text "4-pole Sallen-Key active anti-aliasing lowpass filters\nUnity gain\nfc = 23.2kHz, Q = 0.707 each\nIf sampling at 44.1kHz, nyquist is 22.05kHz\nMust filter hard just below this\n"
+	(text "4-pole Sallen-Key active anti-aliasing lowpass filters\nUnity gain\nfc = 23.2kHz, Q = 0.707 each\nIf sampling at 44.1kHz, nyquist is 22.05kHz\nMust filter hard around this frequency"
 		(exclude_from_sim no)
 		(at 134.62 151.13 0)

Commit message: Annotated schematic
Parts:
- renumbered C71 to C1601, C72 to C1602, C73 to C1603, C74 to C1604, C75 to C1605, C76 to C1606, C77 to C1607, C78 to C1608, C79 to C1609, C80 to C1610, R73 to R1601, R74 to R1602, R75 to R1603, R76 to R1604, R77 to R1605, R78 to R1606, R79 to R1607, R80 to R1608, U26 to U1601

Commit message: cleared stale digikey part numbers
Parts:
- C1601, C1602, C1605, C1606, C1607, C1608: Digi-Key PN 490-10697-1-ND -> (none)
- C1603, C1604, C1609, C1610: footprint (none) -> Capacitors_SMD:C_0402; Digi-Key PN PN -> (none)
- R1601, R1602, R1603, R1604, R1605, R1606, R1607, R1608: Digi-Key PN 541-1.00KHCT-ND -> (none)
Changed lines of the file:
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@@
 			)
 		)
-		(property "Footprint" ""
+		(property "Footprint" "Capacitors_SMD:C_0402"
 			(at 123.19 99.3648 0)
 			(hide yes)
@@
 			)
 		)
-		(property "Digi-Key PN" "PN"
+		(property "Digi-Key PN" ""
 			(at 106.68 89.535 0)
 			(hide yes)
@@
 			)
 		)
-		(property "Digi-Key PN" "490-10697-1-ND"
+		(property "Digi-Key PN" ""
 			(at 90.805 59.69 0)
 			(hide yes)
@@
 			)
 		)
-		(property "Footprint" ""
+		(property "Footprint" "Capacitors_SMD:C_0402"
 			(at 123.19 48.5648 0)
 			(hide yes)
@@
 			)
 		)
-		(property "Digi-Key PN" "PN"
+		(property "Digi-Key PN" ""
 			(at 106.68 38.735 0)
 			(hide yes)
@@
 			)
 		)
-		(property "Digi-Key PN" "541-1.00KHCT-ND"
+		(property "Digi-Key PN" ""
 			(at 163.83 71.12 0)
 			(hide yes)
@@
 			)
 		)
-		(property "Digi-Key PN" "541-1.00KHCT-ND"
+		(property "Digi-Key PN" ""
 			(at 101.6 71.12 0)
 			(hide yes)
@@
 			)
 		)
-		(property "Digi-Key PN" "490-10697-1-ND"
+		(property "Digi-Key PN" ""
 			(at 153.035 59.69 0)
 			(hide yes)
@@
 			)
 		)
-		(property "Digi-Key PN" "541-1.00KHCT-ND"
+		(property "Digi-Key PN" ""
 			(at 88.9 71.12 0)
 			(hide yes)
@@
 			)
 		)
-		(property "Digi-Key PN" "490-10697-1-ND"
+		(property "Digi-Key PN" ""
 			(at 153.035 110.49 0)
 			(hide yes)
@@
 			)
 		)
-		(property "Digi-Key PN" "541-1.00KHCT-ND"
+		(property "Digi-Key PN" ""
 			(at 88.9 121.92 0)
 			(hide yes)
@@
 			)
 		)
-		(property "Digi-Key PN" "541-1.00KHCT-ND"
+		(property "Digi-Key PN" ""
 			(at 151.13 71.12 0)
 			(hide yes)
@@
 			)
 		)
-		(property "Digi-Key PN" "541-1.00KHCT-ND"
+		(property "Digi-Key PN" ""
 			(at 151.13 121.92 0)
 			(hide yes)
@@
 			)
 		)
-		(property "Digi-Key PN" "541-1.00KHCT-ND"
+		(property "Digi-Key PN" ""
 			(at 163.83 121.92 0)
 			(hide yes)
@@
 			)
 		)
-		(property "Digi-Key PN" "541-1.00KHCT-ND"
+		(property "Digi-Key PN" ""
 			(at 101.6 121.92 0)
 			(hide yes)
@@
 			)
 		)
-		(property "Footprint" ""
+		(property "Footprint" "Capacitors_SMD:C_0402"
 			(at 185.42 99.3648 0)
 			(hide yes)
@@
 			)
 		)
-		(property "Digi-Key PN" "PN"
+		(property "Digi-Key PN" ""
 			(at 168.91 89.535 0)
 			(hide yes)
@@
 			)
 		)
-		(property "Digi-Key PN" "490-10697-1-ND"
+		(property "Digi-Key PN" ""
 			(at 126.365 21.59 0)
 			(hide yes)
@@
 			)
 		)
-		(property "Footprint" ""
+		(property "Footprint" "Capacitors_SMD:C_0402"
 			(at 185.42 48.5648 0)
 			(hide yes)
@@
 			)
 		)
-		(property "Digi-Key PN" "PN"
+		(property "Digi-Key PN" ""
 			(at 168.91 38.735 0)
 			(hide yes)
@@
 			)
 		)
-		(property "Digi-Key PN" "490-10697-1-ND"
+		(property "Digi-Key PN" ""
 			(at 90.805 110.49 0)
 			(hide yes)
@@
 			)
 		)
-		(property "Digi-Key PN" "490-10697-1-ND"
+		(property "Digi-Key PN" ""
 			(at 144.145 21.59 0)
 			(hide yes)
