File: hdw/DSP_board/rev_a/Audio_Visualiser_DSP/dspic33_programming.kicad_sch (KiCad schematic)
At the start: 17 parts

Commit message: added a bunch of schematic shit
Parts:
- added C1101: 0.1uF, Capacitors_SMD:C_0603, symbol Custom_Library:C_Custom
- added C?: 10uF, symbol Custom Library:C_Custom
- added C?: 0.1uF, symbol Custom Library:C_Custom
- added FB?: 220, symbol Custom Library:FB_Custom
- added R?: 10, symbol Custom_Library:R_Custom
- added R? (x3): 10k, Resistors_SMD:R_0402, symbol Custom_Library:R_Custom
- added TP1101: TP, Custom Footprints Library:Test_Point, symbol Custom_Library:TP
- added U1101: 74LVC1G97, Package_TO_SOT_SMD:SOT-363_SC-70-6, symbol Custom_Library:74LVC1G97_Power_BUF
- added X1101: ASE-8.000MHz, Oscillator:Oscillator_SMD_Abracon_ASE-4Pin_3.2x2.5mm, symbol Oscillator:ASE-xxxMHz
- R? (x3): footprint Resistors_SMD:R_0603 -> Resistors_SMD:R_0402
- R? (x2): footprint Resistors_SMD:R_0603 -> (none)
Connections:
- net +3.3V: now also C1101.1, FB?.1, U1101.5 (VCC)
- net GND: now also C1101.2, C?.2, C?.2, R?.2, R?.2, R?.2, U1101.2 (GND), U1101.3 (GND), U1101.6 (GND), X1101.2 (GND)
- new net: R?.1, R?.1, X1101.3 (OUT)
- new net: C?.1, C?.1, FB?.2, X1101.4 (Vdd)
- new net DSPIC33_CLK_EN: R?.1, U1101.4, X1101.1 (EN)
- new net DSPIC33_POSC_EC: R?.2
- new net DSPIC33_REFCLK1: R?.1, TP1101.1 (TP)
- new net POS3P3_PGOOD: U1101.1

Commit message: added a ton of circuitry in schematic, new USB UART bridge, other random stuff
Parts:
- renumbered C1101 to C?, TP1101 to TP?, U1101 to U?, X1101 to X?
Other:
- company: Drew Maatman -> (none)
- title: Nixie Clock Redux Core Board -> (none)
Changed lines of the file:
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@@
 	(paper "A")
 	(title_block
-		(title "Nixie Clock Redux Core Board")
 		(date "2023-12-25")
-		(rev "B")
-		(company "Drew Maatman")
 	)
 	(junction
@@
 	)
 	(global_label "~{DSPIC33_MCLR}"
-		(shape passive)
+		(shape output)
 		(at 96.52 33.02 0)
 		(fields_autoplaced yes)
@@
 		)
 		(property "Intersheetrefs" "${INTERSHEET_REFS}"
-			(at 112.4243 33.02 0)
+			(at 113.5356 33.02 0)
 			(hide yes)
 			(show_name no)
@@
 		(in_pos_files yes)
 		(dnp no)
-		(property "Reference" "#PWR039"
+		(property "Reference" "#PWR?"
 			(at 72.39 119.38 0)
 			(hide yes)
@@
 			(project "Audio_Visualiser_DSP"
 				(path "/97a4dfb8-0e16-46f1-9709-8d2007dd0cd3/3d6836fb-edea-466f-ab73-f835ba2b7cb8"
-					(reference "#PWR039")
+					(reference "#PWR?")
 					(unit 1)
 				)
@@
 		(in_pos_files yes)
 		(dnp no)
-		(property "Reference" "#PWR048"
+		(property "Reference" "#PWR?"
 			(at 190.5 125.73 0)
 			(hide yes)
@@
 			(project "Audio_Visualiser_DSP"
 				(path "/97a4dfb8-0e16-46f1-9709-8d2007dd0cd3/3d6836fb-edea-466f-ab73-f835ba2b7cb8"
-					(reference "#PWR048")
+					(reference "#PWR?")
 					(unit 1)
 				)
@@
 		(in_pos_files yes)
 		(dnp no)
-		(property "Reference" "#PWR036"
+		(property "Reference" "#PWR?"
 			(at 69.85 92.71 0)
 			(hide yes)
@@
 			(project "Audio_Visualiser_DSP"
 				(path "/97a4dfb8-0e16-46f1-9709-8d2007dd0cd3/3d6836fb-edea-466f-ab73-f835ba2b7cb8"
-					(reference "#PWR036")
+					(reference "#PWR?")
 					(unit 1)
 				)
@@
 		(in_pos_files yes)
 		(dnp no)
-		(property "Reference" "#PWR041"
+		(property "Reference" "#PWR?"
 			(at 93.98 127 0)
 			(hide yes)
@@
 			(project "Audio_Visualiser_DSP"
 				(path "/97a4dfb8-0e16-46f1-9709-8d2007dd0cd3/3d6836fb-edea-466f-ab73-f835ba2b7cb8"
-					(reference "#PWR041")
+					(reference "#PWR?")
 					(unit 1)
 				)
@@
 		(in_pos_files yes)
 		(dnp no)
-		(property "Reference" "TP1101"
+		(property "Reference" "TP?"
 			(at 97.79 172.72 90)
 			(show_name no)
@@
 			(project "Audio_Visualiser_DSP"
 				(path "/97a4dfb8-0e16-46f1-9709-8d2007dd0cd3/3d6836fb-edea-466f-ab73-f835ba2b7cb8"
-					(reference "TP1101")
+					(reference "TP?")
 					(unit 1)
 				)
@@
 		(in_pos_files yes)
 		(dnp no)
-		(property "Reference" "#PWR040"
+		(property "Reference" "#PWR?"
 			(at 92.71 187.96 0)
 			(hide yes)
@@
 			(project "Audio_Visualiser_DSP"
 				(path "/97a4dfb8-0e16-46f1-9709-8d2007dd0cd3/3d6836fb-edea-466f-ab73-f835ba2b7cb8"
-					(reference "#PWR040")
+					(reference "#PWR?")
 					(unit 1)
 				)
@@
 		(in_pos_files yes)
 		(dnp no)
-		(property "Reference" "#PWR038"
+		(property "Reference" "#PWR?"
 			(at 72.39 111.76 0)
 			(hide yes)
@@
 			(project "Audio_Visualiser_DSP"
 				(path "/97a4dfb8-0e16-46f1-9709-8d2007dd0cd3/3d6836fb-edea-466f-ab73-f835ba2b7cb8"
-					(reference "#PWR038")
+					(reference "#PWR?")
 					(unit 1)
 				)
@@
 		(in_pos_files yes)
 		(dnp no)
-		(property "Reference" "#PWR042"
+		(property "Reference" "#PWR?"
 			(at 137.16 90.17 0)
 			(hide yes)
@@
 			(project "Audio_Visualiser_DSP"
 				(path "/97a4dfb8-0e16-46f1-9709-8d2007dd0cd3/3d6836fb-edea-466f-ab73-f835ba2b7cb8"
-					(reference "#PWR042")
+					(reference "#PWR?")
 					(unit 1)
 				)
@@
 		(in_pos_files yes)
 		(dnp no)
-		(property "Reference" "X1101"
+		(property "Reference" "X?"
 			(at 157.48 104.14 0)
 			(show_name no)
@@
 			(project "Audio_Visualiser_DSP"
 				(path "/97a4dfb8-0e16-46f1-9709-8d2007dd0cd3/3d6836fb-edea-466f-ab73-f835ba2b7cb8"
-					(reference "X1101")
+					(reference "X?")
 					(unit 1)
 				)
@@
 		(in_pos_files yes)
 		(dnp no)
-		(property "Reference" "U1101"
+		(property "Reference" "U?"
 			(at 73.914 106.68 0)
 			(show_name no)
@@
 			(project "Audio_Visualiser_DSP"
 				(path "/97a4dfb8-0e16-46f1-9709-8d2007dd0cd3/3d6836fb-edea-466f-ab73-f835ba2b7cb8"
-					(reference "U1101")
+					(reference "U?")
 					(unit 1)
 				)
@@
 		(in_pos_files yes)
 		(dnp no)
-		(property "Reference" "#PWR044"
+		(property "Reference" "#PWR?"
 			(at 162.56 124.46 0)
 			(hide yes)
@@
 			(project "Audio_Visualiser_DSP"
 				(path "/97a4dfb8-0e16-46f1-9709-8d2007dd0cd3/3d6836fb-edea-466f-ab73-f835ba2b7cb8"
-					(reference "#PWR044")
+					(reference "#PWR?")
 					(unit 1)
 				)
@@
 		(in_pos_files yes)
 		(dnp no)
-		(property "Reference" "#PWR037"
+		(property "Reference" "#PWR?"
 			(at 69.85 102.87 0)
 			(hide yes)
@@
 			(project "Audio_Visualiser_DSP"
 				(path "/97a4dfb8-0e16-46f1-9709-8d2007dd0cd3/3d6836fb-edea-466f-ab73-f835ba2b7cb8"
-					(reference "#PWR037")
+					(reference "#PWR?")
 					(unit 1)
 				)
@@
 		(in_pos_files yes)
 		(dnp no)
-		(property "Reference" "#FLG01101"
+		(property "Reference" "#FLG?"
 			(at 162.56 84.455 0)
 			(hide yes)
@@
 			(project "Audio_Visualiser_DSP"
 				(path "/97a4dfb8-0e16-46f1-9709-8d2007dd0cd3/3d6836fb-edea-466f-ab73-f835ba2b7cb8"
-					(reference "#FLG01101")
+					(reference "#FLG?")
 					(unit 1)
 				)
@@
 		(in_pos_files yes)
 		(dnp no)
-		(property "Reference" "#PWR046"
+		(property "Reference" "#PWR?"
 			(at 177.8 104.14 0)
 			(hide yes)
@@
 			(project "Audio_Visualiser_DSP"
 				(path "/97a4dfb8-0e16-46f1-9709-8d2007dd0cd3/3d6836fb-edea-466f-ab73-f835ba2b7cb8"
-					(reference "#PWR046")
+					(reference "#PWR?")
 					(unit 1)
 				)
@@
 		(in_pos_files yes)
 		(dnp no)
-		(property "Reference" "#PWR050"
+		(property "Reference" "#PWR?"
 			(at 195.58 104.14 0)
 			(hide yes)
@@
 			(project "Audio_Visualiser_DSP"
 				(path "/97a4dfb8-0e16-46f1-9709-8d2007dd0cd3/3d6836fb-edea-466f-ab73-f835ba2b7cb8"
-					(reference "#PWR050")
+					(reference "#PWR?")
 					(unit 1)
 				)
@@
 		(in_pos_files yes)
 		(dnp no)
-		(property "Reference" "C1101"
+		(property "Reference" "C?"
 			(at 69.215 90.17 0)
 			(show_name no)
@@
 			(project "Audio_Visualiser_DSP"
 				(path "/97a4dfb8-0e16-46f1-9709-8d2007dd0cd3/3d6836fb-edea-466f-ab73-f835ba2b7cb8"
-					(reference "C1101")
+					(reference "C?")
 					(unit 1)
 				)

Commit message: Added some spice models
Parts:
- gave numbers to parts that had none: 24

Commit message: added rotary encoder circuitry
Other:
- moved on the sheet: C16, FB1, FB2

Commit message: Annotated schematic
Parts:
- renumbered C15 to C601, C16 to C602, C17 to C603, C18 to C604, C19 to C605, D3 to D601, FB1 to FB601, FB2 to FB602, FB3 to FB603, J2 to J601, Q3 to Q601, R22 to R601, R23 to R602, R24 to R603, R25 to R604, R26 to R605, R27 to R606, R28 to R607, R29 to R608, R30 to R609, SW1 to SW601, TP5 to TP601, U6 to U601, X1 to X601

Commit message: cleared stale digikey part numbers
Parts:
- C601, C602, C605: footprint Capacitors_SMD:C_0603 -> Capacitors_SMD:C_0402; Digi-Key PN 1276-1935-1-ND -> (none)
- C603: footprint (none) -> Capacitors_SMD:C_0402; Digi-Key PN PN -> (none)
- C604: footprint (none) -> Capacitors_SMD:C_0805; Digi-Key PN PN -> (none)
- R601, R602, R604, R605, R608: Digi-Key PN 541-10.0KHCT-ND -> (none)
- R603, R606, R607: footprint (none) -> Resistors_SMD:R_0402; Digi-Key PN 541-10.0HCT-ND -> (none)
- R609: Digi-Key PN 541-1.00KHCT-ND -> (none)
Changed lines of the file:
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@@
 			)
 		)
-		(property "Footprint" ""
+		(property "Footprint" "Resistors_SMD:R_0402"
 			(at 200.66 110.49 0)
 			(hide yes)
@@
 			)
 		)
-		(property "Digi-Key PN" "541-10.0HCT-ND"
+		(property "Digi-Key PN" ""
 			(at 190.5 102.87 0)
 			(hide yes)
@@
 			)
 		)
-		(property "Footprint" "Capacitors_SMD:C_0603"
+		(property "Footprint" "Capacitors_SMD:C_0402"
 			(at 230.8352 50.8 0)
 			(hide yes)
@@
 			)
 		)
-		(property "Digi-Key PN" "1276-1935-1-ND"
+		(property "Digi-Key PN" ""
 			(at 240.665 34.29 0)
 			(hide yes)
@@
 			)
 		)
-		(property "Footprint" ""
+		(property "Footprint" "Capacitors_SMD:C_0805"
 			(at 196.5452 97.79 0)
 			(hide yes)
@@
 			)
 		)
-		(property "Digi-Key PN" "PN"
+		(property "Digi-Key PN" ""
 			(at 206.375 81.28 0)
 			(hide yes)
@@
 			)
 		)
-		(property "Digi-Key PN" "541-1.00KHCT-ND"
+		(property "Digi-Key PN" ""
 			(at 252.73 40.64 0)
 			(hide yes)
@@
 			)
 		)
-		(property "Digi-Key PN" "541-10.0KHCT-ND"
+		(property "Digi-Key PN" ""
 			(at 222.25 16.51 0)
 			(hide yes)
@@
 			)
 		)
-		(property "Footprint" ""
+		(property "Footprint" "Resistors_SMD:R_0402"
 			(at 212.09 33.02 0)
 			(hide yes)
@@
 			)
 		)
-		(property "Digi-Key PN" "541-10.0HCT-ND"
+		(property "Digi-Key PN" ""
 			(at 201.93 25.4 0)
 			(hide yes)
@@
 			)
 		)
-		(property "Footprint" ""
+		(property "Footprint" "Capacitors_SMD:C_0402"
 			(at 178.7652 97.79 0)
 			(hide yes)
@@
 			)
 		)
-		(property "Digi-Key PN" "PN"
+		(property "Digi-Key PN" ""
 			(at 188.595 81.28 0)
 			(hide yes)
@@
 			)
 		)
-		(property "Digi-Key PN" "541-10.0KHCT-ND"
+		(property "Digi-Key PN" ""
 			(at 101.6 106.68 0)
 			(hide yes)
@@
 			)
 		)
-		(property "Footprint" ""
+		(property "Footprint" "Resistors_SMD:R_0402"
 			(at 176.53 45.72 0)
 			(hide yes)
@@
 			)
 		)
-		(property "Digi-Key PN" "541-10.0HCT-ND"
+		(property "Digi-Key PN" ""
 			(at 166.37 38.1 0)
 			(hide yes)
@@
 			)
 		)
-		(property "Digi-Key PN" "541-10.0KHCT-ND"
+		(property "Digi-Key PN" ""
 			(at 198.12 105.41 0)
 			(hide yes)
@@
 			)
 		)
-		(property "Footprint" "Capacitors_SMD:C_0603"
+		(property "Footprint" "Capacitors_SMD:C_0402"
 			(at 120.3452 40.64 0)
 			(hide yes)
@@
 			)
 		)
-		(property "Digi-Key PN" "1276-1935-1-ND"
+		(property "Digi-Key PN" ""
 			(at 130.175 24.13 0)
 			(hide yes)
@@
 			)
 		)
-		(property "Digi-Key PN" "541-10.0KHCT-ND"
+		(property "Digi-Key PN" ""
 			(at 100.33 167.64 0)
 			(hide yes)
@@
 			)
 		)
-		(property "Digi-Key PN" "541-10.0KHCT-ND"
+		(property "Digi-Key PN" ""
 			(at 195.58 41.91 0)
 			(hide yes)
@@
 			)
 		)
-		(property "Footprint" "Capacitors_SMD:C_0603"
+		(property "Footprint" "Capacitors_SMD:C_0402"
 			(at 68.8848 96.52 0)
 			(hide yes)
@@
 			)
 		)
-		(property "Digi-Key PN" "1276-1935-1-ND"
+		(property "Digi-Key PN" ""
 			(at 59.055 80.01 0)
 			(hide yes)

Commit message: updated rca jack
Parts:
- FB601, FB602, FB603: footprint (none) -> Inductors_SMD:L_0402
Changed lines of the file:
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@@
 			)
 		)
-		(property "Footprint" ""
+		(property "Footprint" "Inductors_SMD:L_0402"
 			(at 149.86 87.63 0)
 			(hide yes)
@@
 			)
 		)
-		(property "Footprint" ""
+		(property "Footprint" "Inductors_SMD:L_0402"
 			(at 60.96 33.02 0)
 			(hide yes)
@@
 			)
 		)
-		(property "Footprint" ""
+		(property "Footprint" "Inductors_SMD:L_0402"
 			(at 60.96 38.1 0)
 			(hide yes)
