File: hdw/DSP_board/rev_a/Audio_Visualiser_DSP/audio_voltage_references.kicad_sch (KiCad schematic)
At the start: 10 parts

Commit message: more schematic progress
Parts:
- removed R?: 10k, Resistors_SMD:R_0402, symbol Custom_Library:R_Custom
Changed lines of the file:
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@@
-	)
-	(junction
-		(at 119.38 127)
-		(diameter 0)
-		(color 0 0 0 0)
 	)
 	(junction
@@
 	(wire
 		(pts
-			(xy 119.38 127) (xy 125.73 127)
+			(xy 113.03 127) (xy 125.73 127)
 		)
 		(stroke
@@
 	(wire
 		(pts
-			(xy 113.03 127) (xy 119.38 127)
+			(xy 144.78 66.04) (xy 140.97 66.04)
 		)
 		(stroke
@@
 	(wire
 		(pts
-			(xy 144.78 66.04) (xy 140.97 66.04)
-		)
-		(stroke
-			(width 0)
-			(type default)
-		)
-	)
-	(wire
-		(pts
 			(xy 119.38 66.04) (xy 119.38 63.5)
-		)
-		(stroke
-			(width 0)
-			(type default)
-		)
-	)
-	(wire
-		(pts
-			(xy 119.38 129.54) (xy 119.38 127)
 		)
 		(stroke
@@
 	)
 	(symbol
-		(lib_id "power:GND")
-		(at 119.38 137.16 0)
-		(unit 1)
-		(body_style 1)
-		(exclude_from_sim no)
-		(in_bom yes)
-		(on_board yes)
-		(in_pos_files yes)
-		(dnp no)
-		(property "Reference" "#PWR?"
-			(at 119.38 143.51 0)
-			(hide yes)
-			(show_name no)
-			(do_not_autoplace no)
-			(effects
-				(font
-					(size 1.27 1.27)
-				)
-			)
-		)
-		(property "Value" "GND"
-			(at 119.38 140.97 0)
-			(show_name no)
-			(do_not_autoplace no)
-			(effects
-				(font
-					(size 1.27 1.27)
-				)
-			)
-		)
-		(property "Footprint" ""
-			(at 119.38 137.16 0)
-			(hide yes)
-			(show_name no)
-			(do_not_autoplace no)
-			(effects
-				(font
-					(size 1.27 1.27)
-				)
-			)
-		)
-		(property "Datasheet" ""
-			(at 119.38 137.16 0)
-			(hide yes)
-			(show_name no)
-			(do_not_autoplace no)
-			(effects
-				(font
-					(size 1.27 1.27)
-				)
-			)
-		)
-		(property "Description" "Power symbol creates a global label with name \"GND\" , ground"
-			(at 119.38 137.16 0)
-			(hide yes)
-			(show_name no)
-			(do_not_autoplace no)
-			(effects
-				(font
-					(size 1.27 1.27)
-				)
-			)
-		)
-		(pin "1"
-		)
-		(instances
-			(project "Audio_Visualiser_DSP"
-				(path "/97a4dfb8-0e16-46f1-9709-8d2007dd0cd3/6411608b-521a-4c33-acf3-00a911578dd5"
-					(reference "#PWR?")
-					(unit 1)
-				)
-			)
-		)
-	)
-	(symbol
 		(lib_id "power:+3.3V")
 		(at 133.35 55.88 0)
@@
 					(unit 1)
 				)
-			)
-		)
-	)
-	(symbol
-		(lib_id "Custom_Library:R_Custom")
-		(at 119.38 133.35 0)
-		(mirror y)
-		(unit 1)
-		(body_style 1)
-		(exclude_from_sim no)
-		(in_bom yes)
-		(on_board yes)
-		(in_pos_files yes)
-		(dnp yes)
-		(property "Reference" "R?"
-			(at 117.602 130.048 0)
-			(show_name no)
-			(do_not_autoplace no)
-			(effects
-				(font
-					(size 1.27 1.27)
-				)
-				(justify left)
-			)
-		)
-		(property "Value" "10k"
-			(at 119.38 133.35 90)
-			(show_name no)
-			(do_not_autoplace no)
-			(effects
-				(font
-					(size 1.27 1.27)
-				)
-			)
-		)
-		(property "Footprint" "Resistors_SMD:R_0402"
-			(at 119.38 133.35 0)
-			(hide yes)
-			(show_name no)
-			(do_not_autoplace no)
-			(effects
-				(font
-					(size 1.27 1.27)
-				)
-			)
-		)
-		(property "Datasheet" ""
-			(at 119.38 133.35 0)
-			(hide yes)
-			(show_name no)
-			(do_not_autoplace no)
-			(effects
-				(font
-					(size 1.27 1.27)
-				)
-			)
-		)
-		(property "Description" ""
-			(at 119.38 133.35 0)
-			(show_name no)
-			(do_not_autoplace no)
-			(effects
-				(font
-					(size 1.27 1.27)
-				)
-			)
-		)
-		(property "display_footprint" "0402"
-			(at 117.602 132.08 0)
-			(show_name no)
-			(do_not_autoplace no)
-			(effects
-				(font
-					(size 1.27 1.27)
-				)
-				(justify left)
-			)
-		)
-		(property "Tolerance" "1%"
-			(at 117.602 134.366 0)
-			(show_name no)
-			(do_not_autoplace no)
-			(effects
-				(font
-					(size 1.27 1.27)
-				)
-				(justify left)
-			)
-		)
-		(property "Wattage" "1/16W"
-			(at 117.602 136.652 0)
-			(show_name no)
-			(do_not_autoplace no)
-			(effects
-				(font
-					(size 1.27 1.27)
-				)
-				(justify left)
-			)
-		)
-		(property "Digi-Key PN" "541-100KHCT-ND"
-			(at 119.38 133.35 0)
-			(hide yes)
-			(show_name no)
-			(do_not_autoplace no)
-			(effects
-				(font
-					(size 1.27 1.27)
-				)
-			)
-		)
-		(pin "1"
-		)
-		(pin "2"
-		)
-		(instances
-			(project "Audio_Visualiser_DSP"
-				(path "/97a4dfb8-0e16-46f1-9709-8d2007dd0cd3/6411608b-521a-4c33-acf3-00a911578dd5"
-					(reference "R?")
-					(unit 1)
-				)

Commit message: Added some spice models
Parts:
- gave numbers to parts that had none: 9

Commit message: more signal chain development and simulation
Parts:
- renumbered R79 to R81
Changed lines of the file:
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@@
 		(in_pos_files yes)
 		(dnp no)
-		(property "Reference" "R79"
+		(property "Reference" "R81"
 			(at 117.602 66.548 0)
 			(show_name no)
@@
 			(project "Audio_Visualiser_DSP"
 				(path "/97a4dfb8-0e16-46f1-9709-8d2007dd0cd3/6411608b-521a-4c33-acf3-00a911578dd5"
-					(reference "R79")
+					(reference "R81")
 					(unit 1)
 				)
@@
 		(in_pos_files yes)
 		(dnp no)
-		(property "Reference" "#PWR0282"
+		(property "Reference" "#PWR0291"
 			(at 162.56 146.05 0)
 			(hide yes)
@@
 			(project "Audio_Visualiser_DSP"
 				(path "/97a4dfb8-0e16-46f1-9709-8d2007dd0cd3/6411608b-521a-4c33-acf3-00a911578dd5"
-					(reference "#PWR0282")
+					(reference "#PWR0291")
 					(unit 1)
 				)
@@
 		(in_pos_files yes)
 		(dnp no)
-		(property "Reference" "#PWR0277"
+		(property "Reference" "#PWR0286"
 			(at 144.78 123.19 0)
 			(hide yes)
@@
 			(project "Audio_Visualiser_DSP"
 				(path "/97a4dfb8-0e16-46f1-9709-8d2007dd0cd3/6411608b-521a-4c33-acf3-00a911578dd5"
-					(reference "#PWR0277")
+					(reference "#PWR0286")
 					(unit 1)
 				)
@@
 		(in_pos_files yes)
 		(dnp no)
-		(property "Reference" "#PWR0271"
+		(property "Reference" "#PWR0280"
 			(at 133.35 123.19 0)
 			(hide yes)
@@
 			(project "Audio_Visualiser_DSP"
 				(path "/97a4dfb8-0e16-46f1-9709-8d2007dd0cd3/6411608b-521a-4c33-acf3-00a911578dd5"
-					(reference "#PWR0271")
+					(reference "#PWR0280")
 					(unit 1)
 				)
@@
 		(dnp no)
 		(fields_autoplaced yes)
-		(property "Reference" "#PWR0281"
+		(property "Reference" "#PWR0290"
 			(at 162.56 128.27 0)
 			(hide yes)
@@
 			(project "Audio_Visualiser_DSP"
 				(path "/97a4dfb8-0e16-46f1-9709-8d2007dd0cd3/6411608b-521a-4c33-acf3-00a911578dd5"
-					(reference "#PWR0281")
+					(reference "#PWR0290")
 					(unit 1)
 				)
@@
 		(in_pos_files yes)
 		(dnp no)
-		(property "Reference" "#PWR0276"
+		(property "Reference" "#PWR0285"
 			(at 144.78 113.03 0)
 			(hide yes)
@@
 			(project "Audio_Visualiser_DSP"
 				(path "/97a4dfb8-0e16-46f1-9709-8d2007dd0cd3/6411608b-521a-4c33-acf3-00a911578dd5"
-					(reference "#PWR0276")
+					(reference "#PWR0285")
 					(unit 1)
 				)
@@
 		(in_pos_files yes)
 		(dnp no)
-		(property "Reference" "#PWR0278"
+		(property "Reference" "#PWR0287"
 			(at 144.78 146.05 0)
 			(hide yes)
@@
 			(project "Audio_Visualiser_DSP"
 				(path "/97a4dfb8-0e16-46f1-9709-8d2007dd0cd3/6411608b-521a-4c33-acf3-00a911578dd5"
-					(reference "#PWR0278")
+					(reference "#PWR0287")
 					(unit 1)
 				)
@@
 		(in_pos_files yes)
 		(dnp no)
-		(property "Reference" "#PWR0273"
+		(property "Reference" "#PWR0282"
 			(at 144.78 49.53 0)
 			(hide yes)
@@
 			(project "Audio_Visualiser_DSP"
 				(path "/97a4dfb8-0e16-46f1-9709-8d2007dd0cd3/6411608b-521a-4c33-acf3-00a911578dd5"
-					(reference "#PWR0273")
+					(reference "#PWR0282")
 					(unit 1)
 				)
@@
 		(in_pos_files yes)
 		(dnp no)
-		(property "Reference" "#PWR0275"
+		(property "Reference" "#PWR0284"
 			(at 144.78 82.55 0)
 			(hide yes)
@@
 			(project "Audio_Visualiser_DSP"
 				(path "/97a4dfb8-0e16-46f1-9709-8d2007dd0cd3/6411608b-521a-4c33-acf3-00a911578dd5"
-					(reference "#PWR0275")
+					(reference "#PWR0284")
 					(unit 1)
 				)
@@
 		(in_pos_files yes)
 		(dnp no)
-		(property "Reference" "#PWR0269"
+		(property "Reference" "#PWR0278"
 			(at 133.35 59.69 0)
 			(hide yes)
@@
 			(project "Audio_Visualiser_DSP"
 				(path "/97a4dfb8-0e16-46f1-9709-8d2007dd0cd3/6411608b-521a-4c33-acf3-00a911578dd5"
-					(reference "#PWR0269")
+					(reference "#PWR0278")
 					(unit 1)
 				)
@@
 		(in_pos_files yes)
 		(dnp no)
-		(property "Reference" "#PWR0272"
+		(property "Reference" "#PWR0281"
 			(at 133.35 140.97 0)
 			(hide yes)
@@
 			(project "Audio_Visualiser_DSP"
 				(path "/97a4dfb8-0e16-46f1-9709-8d2007dd0cd3/6411608b-521a-4c33-acf3-00a911578dd5"
-					(reference "#PWR0272")
+					(reference "#PWR0281")
 					(unit 1)
 				)
@@
 		(in_pos_files yes)
 		(dnp no)
-		(property "Reference" "#PWR0280"
+		(property "Reference" "#PWR0289"
 			(at 162.56 82.55 0)
 			(hide yes)
@@
 			(project "Audio_Visualiser_DSP"
 				(path "/97a4dfb8-0e16-46f1-9709-8d2007dd0cd3/6411608b-521a-4c33-acf3-00a911578dd5"
-					(reference "#PWR0280")
+					(reference "#PWR0289")
 					(unit 1)
 				)
@@
 		(dnp no)
 		(fields_autoplaced yes)
-		(property "Reference" "#PWR0279"
+		(property "Reference" "#PWR0288"
 			(at 162.56 64.77 0)
 			(hide yes)
@@
 			(project "Audio_Visualiser_DSP"
 				(path "/97a4dfb8-0e16-46f1-9709-8d2007dd0cd3/6411608b-521a-4c33-acf3-00a911578dd5"
-					(reference "#PWR0279")
+					(reference "#PWR0288")
 					(unit 1)
 				)
@@
 		(in_pos_files yes)
 		(dnp no)
-		(property "Reference" "#PWR0268"
+		(property "Reference" "#PWR0277"
 			(at 119.38 80.01 0)
 			(hide yes)
@@
 			(project "Audio_Visualiser_DSP"
 				(path "/97a4dfb8-0e16-46f1-9709-8d2007dd0cd3/6411608b-521a-4c33-acf3-00a911578dd5"
-					(reference "#PWR0268")
+					(reference "#PWR0277")
 					(unit 1)
 				)
@@
 		(in_pos_files yes)
 		(dnp no)
-		(property "Reference" "#PWR0274"
+		(property "Reference" "#PWR0283"
 			(at 144.78 59.69 0)
 			(hide yes)
@@
 			(project "Audio_Visualiser_DSP"
 				(path "/97a4dfb8-0e16-46f1-9709-8d2007dd0cd3/6411608b-521a-4c33-acf3-00a911578dd5"
-					(reference "#PWR0274")
+					(reference "#PWR0283")
 					(unit 1)
 				)
@@
 		(in_pos_files yes)
 		(dnp no)
-		(property "Reference" "#PWR0270"
+		(property "Reference" "#PWR0279"
 			(at 133.35 77.47 0)
 			(hide yes)
@@
 			(project "Audio_Visualiser_DSP"
 				(path "/97a4dfb8-0e16-46f1-9709-8d2007dd0cd3/6411608b-521a-4c33-acf3-00a911578dd5"
-					(reference "#PWR0270")
-					(unit 1)
-				)
+					(reference "#PWR0279")
+					(unit 1)
+				)

Commit message: Annotated schematic
Parts:
- renumbered C81 to C1701, C82 to C1702, C83 to C1703, C84 to C1704, C85 to C1705, C86 to C1706, R81 to R1701, U27 to U1701, U28 to U1702
Changed lines of the file:
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@@
 		(in_pos_files yes)
 		(dnp no)
-		(property "Reference" "R81"
+		(property "Reference" "R1701"
 			(at 117.602 66.548 0)
 			(show_name no)
@@
 			(project "Audio_Visualiser_DSP"
 				(path "/97a4dfb8-0e16-46f1-9709-8d2007dd0cd3/6411608b-521a-4c33-acf3-00a911578dd5"
-					(reference "R81")
+					(reference "R1701")
 					(unit 1)
 				)
@@
 		(in_pos_files yes)
 		(dnp no)
-		(property "Reference" "C82"
+		(property "Reference" "C1702"
 			(at 144.145 69.85 0)
 			(show_name no)
@@
 			(project "Audio_Visualiser_DSP"
 				(path "/97a4dfb8-0e16-46f1-9709-8d2007dd0cd3/6411608b-521a-4c33-acf3-00a911578dd5"
-					(reference "C82")
+					(reference "C1702")
 					(unit 1)
 				)
@@
 		(in_pos_files yes)
 		(dnp no)
-		(property "Reference" "#PWR0291"
+		(property "Reference" "#PWR01715"
 			(at 162.56 146.05 0)
 			(hide yes)
@@
 			(project "Audio_Visualiser_DSP"
 				(path "/97a4dfb8-0e16-46f1-9709-8d2007dd0cd3/6411608b-521a-4c33-acf3-00a911578dd5"
-					(reference "#PWR0291")
+					(reference "#PWR01715")
 					(unit 1)
 				)
@@
 		(in_pos_files yes)
 		(dnp no)
-		(property "Reference" "#PWR0286"
+		(property "Reference" "#PWR01710"
 			(at 144.78 123.19 0)
 			(hide yes)
@@
 			(project "Audio_Visualiser_DSP"
 				(path "/97a4dfb8-0e16-46f1-9709-8d2007dd0cd3/6411608b-521a-4c33-acf3-00a911578dd5"
-					(reference "#PWR0286")
+					(reference "#PWR01710")
 					(unit 1)
 				)
@@
 		(in_pos_files yes)
 		(dnp no)
-		(property "Reference" "#PWR0280"
+		(property "Reference" "#PWR01704"
 			(at 133.35 123.19 0)
 			(hide yes)
@@
 			(project "Audio_Visualiser_DSP"
 				(path "/97a4dfb8-0e16-46f1-9709-8d2007dd0cd3/6411608b-521a-4c33-acf3-00a911578dd5"
-					(reference "#PWR0280")
+					(reference "#PWR01704")
 					(unit 1)
 				)
@@
 		(in_pos_files yes)
 		(dnp no)
-		(property "Reference" "C84"
+		(property "Reference" "C1704"
 			(at 144.145 133.35 0)
 			(show_name no)
@@
 			(project "Audio_Visualiser_DSP"
 				(path "/97a4dfb8-0e16-46f1-9709-8d2007dd0cd3/6411608b-521a-4c33-acf3-00a911578dd5"
-					(reference "C84")
+					(reference "C1704")
 					(unit 1)
 				)
@@
 		(dnp no)
 		(fields_autoplaced yes)
-		(property "Reference" "#PWR0290"
+		(property "Reference" "#PWR01714"
 			(at 162.56 128.27 0)
 			(hide yes)
@@
 			(project "Audio_Visualiser_DSP"
 				(path "/97a4dfb8-0e16-46f1-9709-8d2007dd0cd3/6411608b-521a-4c33-acf3-00a911578dd5"
-					(reference "#PWR0290")
+					(reference "#PWR01714")
 					(unit 1)
 				)
@@
 		(in_pos_files yes)
 		(dnp no)
-		(property "Reference" "#PWR0285"
+		(property "Reference" "#PWR01709"
 			(at 144.78 113.03 0)
 			(hide yes)
@@
 			(project "Audio_Visualiser_DSP"
 				(path "/97a4dfb8-0e16-46f1-9709-8d2007dd0cd3/6411608b-521a-4c33-acf3-00a911578dd5"
-					(reference "#PWR0285")
+					(reference "#PWR01709")
 					(unit 1)
 				)
@@
 		(in_pos_files yes)
 		(dnp no)
-		(property "Reference" "#PWR0287"
+		(property "Reference" "#PWR01711"
 			(at 144.78 146.05 0)
 			(hide yes)
@@
 			(project "Audio_Visualiser_DSP"
 				(path "/97a4dfb8-0e16-46f1-9709-8d2007dd0cd3/6411608b-521a-4c33-acf3-00a911578dd5"
-					(reference "#PWR0287")
+					(reference "#PWR01711")
 					(unit 1)
 				)
@@
 		(in_pos_files yes)
 		(dnp no)
-		(property "Reference" "#PWR0282"
+		(property "Reference" "#PWR01706"
 			(at 144.78 49.53 0)
 			(hide yes)
@@
 			(project "Audio_Visualiser_DSP"
 				(path "/97a4dfb8-0e16-46f1-9709-8d2007dd0cd3/6411608b-521a-4c33-acf3-00a911578dd5"
-					(reference "#PWR0282")
+					(reference "#PWR01706")
 					(unit 1)
 				)
@@
 		(in_pos_files yes)
 		(dnp no)
-		(property "Reference" "#PWR0284"
+		(property "Reference" "#PWR01708"
 			(at 144.78 82.55 0)
 			(hide yes)
@@
 			(project "Audio_Visualiser_DSP"
 				(path "/97a4dfb8-0e16-46f1-9709-8d2007dd0cd3/6411608b-521a-4c33-acf3-00a911578dd5"
-					(reference "#PWR0284")
+					(reference "#PWR01708")
 					(unit 1)
 				)
@@
 		(in_pos_files yes)
 		(dnp no)
-		(property "Reference" "#PWR0278"
+		(property "Reference" "#PWR01702"
 			(at 133.35 59.69 0)
 			(hide yes)
@@
 			(project "Audio_Visualiser_DSP"
 				(path "/97a4dfb8-0e16-46f1-9709-8d2007dd0cd3/6411608b-521a-4c33-acf3-00a911578dd5"
-					(reference "#PWR0278")
+					(reference "#PWR01702")
 					(unit 1)
 				)
@@
 		(in_pos_files yes)
 		(dnp no)
-		(property "Reference" "#PWR0281"
+		(property "Reference" "#PWR01705"
 			(at 133.35 140.97 0)
 			(hide yes)
@@
 			(project "Audio_Visualiser_DSP"
 				(path "/97a4dfb8-0e16-46f1-9709-8d2007dd0cd3/6411608b-521a-4c33-acf3-00a911578dd5"
-					(reference "#PWR0281")
+					(reference "#PWR01705")
 					(unit 1)
 				)
@@
 		(dnp no)
 		(fields_autoplaced yes)
-		(property "Reference" "U28"
+		(property "Reference" "U1702"
 			(at 119.38 120.5798 0)
 			(show_name no)
@@
 			(project "Audio_Visualiser_DSP"
 				(path "/97a4dfb8-0e16-46f1-9709-8d2007dd0cd3/6411608b-521a-4c33-acf3-00a911578dd5"
-					(reference "U28")
+					(reference "U1702")
 					(unit 1)
 				)
@@
 		(dnp no)
 		(fields_autoplaced yes)
-		(property "Reference" "U27"
+		(property "Reference" "U1701"
 			(at 119.38 57.0798 0)
 			(show_name no)
@@
 			(project "Audio_Visualiser_DSP"
 				(path "/97a4dfb8-0e16-46f1-9709-8d2007dd0cd3/6411608b-521a-4c33-acf3-00a911578dd5"
-					(reference "U27")
+					(reference "U1701")
 					(unit 1)
 				)
@@
 		(in_pos_files yes)
 		(dnp no)
-		(property "Reference" "#PWR0289"
+		(property "Reference" "#PWR01713"
 			(at 162.56 82.55 0)
 			(hide yes)
@@
 			(project "Audio_Visualiser_DSP"
 				(path "/97a4dfb8-0e16-46f1-9709-8d2007dd0cd3/6411608b-521a-4c33-acf3-00a911578dd5"
-					(reference "#PWR0289")
+					(reference "#PWR01713")
 					(unit 1)
 				)
@@
 		(in_pos_files yes)
 		(dnp no)
-		(property "Reference" "C85"
+		(property "Reference" "C1705"
 			(at 161.925 69.85 0)
 			(show_name no)
@@
 			(project "Audio_Visualiser_DSP"
 				(path "/97a4dfb8-0e16-46f1-9709-8d2007dd0cd3/6411608b-521a-4c33-acf3-00a911578dd5"
-					(reference "C85")
+					(reference "C1705")
 					(unit 1)
 				)
@@
 		(dnp no)
 		(fields_autoplaced yes)
-		(property "Reference" "#PWR0288"
+		(property "Reference" "#PWR01712"
 			(at 162.56 64.77 0)
 			(hide yes)
@@
 			(project "Audio_Visualiser_DSP"
 				(path "/97a4dfb8-0e16-46f1-9709-8d2007dd0cd3/6411608b-521a-4c33-acf3-00a911578dd5"
-					(reference "#PWR0288")
+					(reference "#PWR01712")
 					(unit 1)
 				)
@@
 		(in_pos_files yes)
 		(dnp no)
-		(property "Reference" "C86"
+		(property "Reference" "C1706"
 			(at 161.925 133.35 0)
 			(show_name no)
@@
 			(project "Audio_Visualiser_DSP"
 				(path "/97a4dfb8-0e16-46f1-9709-8d2007dd0cd3/6411608b-521a-4c33-acf3-00a911578dd5"
-					(reference "C86")
+					(reference "C1706")
 					(unit 1)
 				)
@@
 		(in_pos_files yes)
 		(dnp no)
-		(property "Reference" "#PWR0277"
+		(property "Reference" "#PWR01701"
 			(at 119.38 80.01 0)
 			(hide yes)
@@
 			(project "Audio_Visualiser_DSP"
 				(path "/97a4dfb8-0e16-46f1-9709-8d2007dd0cd3/6411608b-521a-4c33-acf3-00a911578dd5"
-					(reference "#PWR0277")
+					(reference "#PWR01701")
 					(unit 1)
 				)
@@
 		(in_pos_files yes)
 		(dnp no)
-		(property "Reference" "#PWR0283"
+		(property "Reference" "#PWR01707"
 			(at 144.78 59.69 0)
 			(hide yes)
@@
 			(project "Audio_Visualiser_DSP"
 				(path "/97a4dfb8-0e16-46f1-9709-8d2007dd0cd3/6411608b-521a-4c33-acf3-00a911578dd5"
-					(reference "#PWR0283")
+					(reference "#PWR01707")
 					(unit 1)
 				)
@@
 		(in_pos_files yes)
 		(dnp no)
-		(property "Reference" "C83"
+		(property "Reference" "C1703"
 			(at 144.145 110.49 0)
 			(show_name no)
@@
 			(project "Audio_Visualiser_DSP"
 				(path "/97a4dfb8-0e16-46f1-9709-8d2007dd0cd3/6411608b-521a-4c33-acf3-00a911578dd5"
-					(reference "C83")
+					(reference "C1703")
 					(unit 1)
 				)
@@
 		(in_pos_files yes)
 		(dnp no)
-		(property "Reference" "C81"
+		(property "Reference" "C1701"
 			(at 144.145 46.99 0)
 			(show_name no)
@@
 			(project "Audio_Visualiser_DSP"
 				(path "/97a4dfb8-0e16-46f1-9709-8d2007dd0cd3/6411608b-521a-4c33-acf3-00a911578dd5"
-					(reference "C81")
+					(reference "C1701")
 					(unit 1)
 				)
@@
 		(in_pos_files yes)
 		(dnp no)
-		(property "Reference" "#PWR0279"
+		(property "Reference" "#PWR01703"
 			(at 133.35 77.47 0)
 			(hide yes)
@@
 			(project "Audio_Visualiser_DSP"
 				(path "/97a4dfb8-0e16-46f1-9709-8d2007dd0cd3/6411608b-521a-4c33-acf3-00a911578dd5"
-					(reference "#PWR0279")
-					(unit 1)
-				)
+					(reference "#PWR01703")
+					(unit 1)
+				)

Commit message: cleared stale digikey part numbers
Parts:
- C1701, C1702, C1703, C1704, C1705, C1706: Digi-Key PN 490-10697-1-ND -> (none)
- R1701: Digi-Key PN 541-100KHCT-ND -> (none)
Changed lines of the file:
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@@
 			)
 		)
-		(property "Digi-Key PN" "541-100KHCT-ND"
+		(property "Digi-Key PN" ""
 			(at 119.38 69.85 0)
 			(hide yes)
@@
 			)
 		)
-		(property "Digi-Key PN" "490-10697-1-ND"
+		(property "Digi-Key PN" ""
 			(at 133.985 59.69 0)
 			(hide yes)
@@
 			)
 		)
-		(property "Digi-Key PN" "490-10697-1-ND"
+		(property "Digi-Key PN" ""
 			(at 133.985 123.19 0)
 			(hide yes)
@@
 			)
 		)
-		(property "Digi-Key PN" "490-10697-1-ND"
+		(property "Digi-Key PN" ""
 			(at 151.765 59.69 0)
 			(hide yes)
@@
 			)
 		)
-		(property "Digi-Key PN" "490-10697-1-ND"
+		(property "Digi-Key PN" ""
 			(at 151.765 123.19 0)
 			(hide yes)
@@
 			)
 		)
-		(property "Digi-Key PN" "490-10697-1-ND"
+		(property "Digi-Key PN" ""
 			(at 133.985 100.33 0)
 			(hide yes)
@@
 			)
 		)
-		(property "Digi-Key PN" "490-10697-1-ND"
+		(property "Digi-Key PN" ""
 			(at 133.985 36.83 0)
 			(hide yes)
