File: hdw/DSP_board/rev_a/Audio_Visualiser_DSP/usb_uart_bridge.kicad_sch (KiCad schematic)
At the start: 32 parts, among them J901 USB_C_Receptacle_USB2.0_14P, U901 CP2104, U902 74LVC1G97, U903 TXB0102YZP, U904 TPD3S014DBVR

Commit message: cleared stale digikey part numbers
Parts:
- C901, C904, C907, C908, C909: footprint Capacitors_SMD:C_0603 -> Capacitors_SMD:C_0402; Digi-Key PN 1276-1935-1-ND -> (none)
- C902, C903, C905, C906, C910: footprint Capacitors_SMD:C_0603 -> Capacitors_SMD:C_0402; Digi-Key PN 1276-1871-1-ND -> (none)
- D903: Digi-Key PN 754-1121-1-ND -> (none)
- R901, R902, R905, R906, R909, R910: Digi-Key PN 541-1.00KHCT-ND -> (none)
- R903, R904, R907, R908: Digi-Key PN 541-100KHCT-ND -> (none)
Changed lines of the file:
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@@
 			)
 		)
-		(property "Digi-Key PN" "541-100KHCT-ND"
+		(property "Digi-Key PN" ""
 			(at 82.55 30.48 0)
 			(hide yes)
@@
 			)
 		)
-		(property "Footprint" "Capacitors_SMD:C_0603"
+		(property "Footprint" "Capacitors_SMD:C_0402"
 			(at 24.4348 156.21 0)
 			(hide yes)
@@
 			)
 		)
-		(property "Digi-Key PN" "1276-1935-1-ND"
+		(property "Digi-Key PN" ""
 			(at 14.605 139.7 0)
 			(hide yes)
@@
 			)
 		)
-		(property "Footprint" "Capacitors_SMD:C_0603"
+		(property "Footprint" "Capacitors_SMD:C_0402"
 			(at 171.1452 59.69 0)
 			(hide yes)
@@
 			)
 		)
-		(property "Digi-Key PN" "1276-1871-1-ND"
+		(property "Digi-Key PN" ""
 			(at 170.18 55.88 0)
 			(hide yes)
@@
 			)
 		)
-		(property "Footprint" "Capacitors_SMD:C_0603"
+		(property "Footprint" "Capacitors_SMD:C_0402"
 			(at 141.9352 87.63 0)
 			(hide yes)
@@
 			)
 		)
-		(property "Digi-Key PN" "1276-1935-1-ND"
+		(property "Digi-Key PN" ""
 			(at 151.765 71.12 0)
 			(hide yes)
@@
 			)
 		)
-		(property "Digi-Key PN" "541-100KHCT-ND"
+		(property "Digi-Key PN" ""
 			(at 177.8 30.48 0)
 			(hide yes)
@@
 			)
 		)
-		(property "Digi-Key PN" "541-1.00KHCT-ND"
+		(property "Digi-Key PN" ""
 			(at 124.46 158.75 0)
 			(hide yes)
@@
 			)
 		)
-		(property "Digi-Key PN" "541-1.00KHCT-ND"
+		(property "Digi-Key PN" ""
 			(at 195.58 114.3 0)
 			(hide yes)
@@
 			)
 		)
-		(property "Footprint" "Capacitors_SMD:C_0603"
+		(property "Footprint" "Capacitors_SMD:C_0402"
 			(at 94.9452 59.69 0)
 			(hide yes)
@@
 			)
 		)
-		(property "Digi-Key PN" "1276-1935-1-ND"
+		(property "Digi-Key PN" ""
 			(at 104.775 43.18 0)
 			(hide yes)
@@
 			)
 		)
-		(property "Footprint" "Capacitors_SMD:C_0603"
+		(property "Footprint" "Capacitors_SMD:C_0402"
 			(at 116.5352 143.51 0)
 			(hide yes)
@@
 			)
 		)
-		(property "Digi-Key PN" "1276-1871-1-ND"
+		(property "Digi-Key PN" ""
 			(at 115.57 139.7 0)
 			(hide yes)
@@
 			)
 		)
-		(property "Footprint" "Capacitors_SMD:C_0603"
+		(property "Footprint" "Capacitors_SMD:C_0402"
 			(at 152.0952 59.69 0)
 			(hide yes)
@@
 			)
 		)
-		(property "Digi-Key PN" "1276-1935-1-ND"
+		(property "Digi-Key PN" ""
 			(at 161.925 43.18 0)
 			(hide yes)
@@
 			)
 		)
-		(property "Digi-Key PN" "541-100KHCT-ND"
+		(property "Digi-Key PN" ""
 			(at 69.85 30.48 0)
 			(hide yes)
@@
 			)
 		)
-		(property "Digi-Key PN" "541-100KHCT-ND"
+		(property "Digi-Key PN" ""
 			(at 190.5 30.48 0)
 			(hide yes)
@@
 			)
 		)
-		(property "Footprint" "Capacitors_SMD:C_0603"
+		(property "Footprint" "Capacitors_SMD:C_0402"
 			(at 114.6048 168.91 0)
 			(hide yes)
@@
 			)
 		)
-		(property "Digi-Key PN" "1276-1935-1-ND"
+		(property "Digi-Key PN" ""
 			(at 104.775 152.4 0)
 			(hide yes)
@@
 			)
 		)
-		(property "Digi-Key PN" "541-1.00KHCT-ND"
+		(property "Digi-Key PN" ""
 			(at 41.91 92.71 0)
 			(hide yes)
@@
 			)
 		)
-		(property "Digi-Key PN" "541-1.00KHCT-ND"
+		(property "Digi-Key PN" ""
 			(at 208.28 114.3 0)
 			(hide yes)
@@
 			)
 		)
-		(property "Digi-Key PN" "541-1.00KHCT-ND"
+		(property "Digi-Key PN" ""
 			(at 29.21 92.71 0)
 			(hide yes)
@@
 			)
 		)
-		(property "Footprint" "Capacitors_SMD:C_0603"
+		(property "Footprint" "Capacitors_SMD:C_0402"
 			(at 113.9952 59.69 0)
 			(hide yes)
@@
 			)
 		)
-		(property "Digi-Key PN" "1276-1871-1-ND"
+		(property "Digi-Key PN" ""
 			(at 113.03 55.88 0)
 			(hide yes)
@@
 			)
 		)
-		(property "Digi-Key PN" "541-1.00KHCT-ND"
+		(property "Digi-Key PN" ""
 			(at 111.76 166.37 0)
 			(hide yes)
@@
 			)
 		)
-		(property "Footprint" "Capacitors_SMD:C_0603"
+		(property "Footprint" "Capacitors_SMD:C_0402"
 			(at 44.7548 156.21 0)
 			(hide yes)
@@
 			)
 		)
-		(property "Digi-Key PN" "1276-1871-1-ND"
+		(property "Digi-Key PN" ""
 			(at 45.72 152.4 0)
 			(hide yes)
@@
 			)
 		)
-		(property "Footprint" "Capacitors_SMD:C_0603"
+		(property "Footprint" "Capacitors_SMD:C_0402"
 			(at 65.0748 156.21 0)
 			(hide yes)
@@
 			)
 		)
-		(property "Digi-Key PN" "1276-1871-1-ND"
+		(property "Digi-Key PN" ""
 			(at 66.04 152.4 0)
 			(hide yes)
@@
 			)
 		)
-		(property "Digi-Key PN" "754-1121-1-ND"
+		(property "Digi-Key PN" ""
 			(at 292.608 307.594 0)
 			(hide yes)

Commit message: updated rca jack
Parts:
- D901, D902: footprint (none) -> LEDs:LED_0402
- D903: footprint LEDs:LED_0603 -> LEDs:LED_0402
- FB901, FB902: footprint (none) -> Inductors_SMD:L_0402
- J901: footprint (none) -> Connector_USB:USB_C_Receptacle_JAE_DX07S016JA1R1500
Changed lines of the file:
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@@
 			)
 		)
-		(property "Footprint" ""
+		(property "Footprint" "LEDs:LED_0402"
 			(at 21.59 110.49 0)
 			(hide yes)
@@
 			)
 		)
-		(property "Footprint" ""
+		(property "Footprint" "Connector_USB:USB_C_Receptacle_JAE_DX07S016JA1R1500"
 			(at 236.22 105.41 0)
 			(hide yes)
@@
 			)
 		)
-		(property "Footprint" ""
+		(property "Footprint" "LEDs:LED_0402"
 			(at 34.29 110.49 0)
 			(hide yes)
@@
 			)
 		)
-		(property "Footprint" ""
+		(property "Footprint" "Inductors_SMD:L_0402"
 			(at 204.47 90.17 0)
 			(hide yes)
@@
 			)
 		)
-		(property "Footprint" ""
+		(property "Footprint" "Inductors_SMD:L_0402"
 			(at 247.65 134.62 0)
 			(hide yes)
@@
 			)
 		)
-		(property "Footprint" "LEDs:LED_0603"
+		(property "Footprint" "LEDs:LED_0402"
 			(at 132.08 176.53 0)
 			(hide yes)

Commit message: assigned some footprints
Parts:
- U901: footprint (none) -> Package_DFN_QFN:QFN-24-1EP_4x4mm_P0.5mm_EP2.65x2.65mm

Commit message: assigned many digi-key part numbers
Parts:
- C901, C904, C907, C908, C909: Digi-Key PN (none) -> 1276-CL05B104KB5NNNCCT-ND
- C902, C903, C905, C906, C910: Digi-Key PN (none) -> 1276-CL05A106MP6NUN8CT-ND
- D901: Digi-Key PN (none) -> 732-11993-1-ND
- D902, D903: Digi-Key PN (none) -> 732-11992-1-ND
- FB901, FB902: Ampacity 0.7A -> 1.3A; Digi-Key PN (none) -> 490-16508-1-ND
- J901: Digi-Key PN (none) -> 670-DX07S016JA1R1500CT-ND
- R901, R902, R906: Digi-Key PN (none) -> 311-1.00KLRCT-ND
- R903, R904, R907, R908: Digi-Key PN (none) -> 311-100KLRCT-ND
- R905, R909, R910: Digi-Key PN (none) -> YAG3503CT-ND
- U903: value TXB0102YZP -> TXB0102DCU; footprint Package_BGA:Texas_DSBGA-8_0.9x1.9mm_Layout2x4_P0.5mm -> Package_SO:VSSOP-8_2.3x2mm_P0.5mm; symbol Logic_LevelTranslator:TXB0102YZP -> Logic_LevelTranslator:TXB0102DCU; Digi-Key PN (none) -> 296-22862-1-ND
Connections:
- net +3.3V: now also U903.7 (VCCB); no longer U903.B2 (VCCB)
- net +3.3V_USB: now also U903.3 (VCCA); no longer U903.C1 (VCCA)
- net GND: now also U903.2 (GND); no longer U903.B1 (GND)
- net USB_UART_RX: now also U903.8 (B1); no longer U903.A2 (B1)
- net USB_UART_RX_BRIDGE: now also U903.5 (A1); no longer U903.D2 (A1)
- net USB_UART_TX: now also U903.1 (B2); no longer U903.A1 (B2)
- net USB_UART_TX_BRIDGE: now also U903.4 (A2); no longer U903.D1 (A2)
- net ~{USB_BRIDGE_RESET}: now also U903.6 (OE); no longer U903.C2 (OE)
Changed lines of the file:
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@@
 			)
 		)
-		(property "Digi-Key PN" ""
+		(property "Digi-Key PN" "311-100KLRCT-ND"
 			(at 82.55 30.48 0)
 			(hide yes)
@@
 			)
 		)
-		(property "Digi-Key PN" ""
+		(property "Digi-Key PN" "732-11993-1-ND"
 			(at 151.638 279.146 0)
 			(hide yes)
@@
 			)
 		)
-		(property "Digi-Key PN" ""
+		(property "Digi-Key PN" "1276-CL05B104KB5NNNCCT-ND"
 			(at 14.605 139.7 0)
 			(hide yes)
@@
 			)
 		)
-		(property "Digi-Key PN" ""
+		(property "Digi-Key PN" "1276-CL05A106MP6NUN8CT-ND"
 			(at 170.18 55.88 0)
 			(hide yes)
@@
 			)
 		)
+		(property "Digi-Key PN" "670-DX07S016JA1R1500CT-ND"
+			(at 240.03 105.41 0)
+			(hide yes)
+			(show_name no)
+			(do_not_autoplace no)
+			(effects
+				(font
+					(size 1.27 1.27)
+				)
+			)
+		)
 		(pin "B6"
 		)
@@
 			)
 		)
-		(property "Digi-Key PN" ""
+		(property "Digi-Key PN" "1276-CL05B104KB5NNNCCT-ND"
 			(at 151.765 71.12 0)
 			(hide yes)
@@
 			)
 		)
-		(property "Digi-Key PN" ""
+		(property "Digi-Key PN" "311-100KLRCT-ND"
 			(at 177.8 30.48 0)
 			(hide yes)
@@
 			)
 		)
-		(property "Digi-Key PN" ""
+		(property "Digi-Key PN" "311-1.00KLRCT-ND"
 			(at 124.46 158.75 0)
 			(hide yes)
@@
 			)
 		)
-		(property "Digi-Key PN" ""
+		(property "Digi-Key PN" "YAG3503CT-ND"
 			(at 195.58 114.3 0)
 			(hide yes)
@@
 			)
 		)
-		(property "Digi-Key PN" ""
+		(property "Digi-Key PN" "1276-CL05B104KB5NNNCCT-ND"
 			(at 104.775 43.18 0)
 			(hide yes)
@@
 			)
 		)
-		(property "Digi-Key PN" ""
+		(property "Digi-Key PN" "1276-CL05A106MP6NUN8CT-ND"
 			(at 115.57 139.7 0)
 			(hide yes)
@@
 			)
 		)
-		(property "Digi-Key PN" ""
+		(property "Digi-Key PN" "732-11992-1-ND"
 			(at 164.338 279.146 0)
 			(hide yes)
@@
 			)
 		)
-		(property "Digi-Key PN" ""
+		(property "Digi-Key PN" "1276-CL05B104KB5NNNCCT-ND"
 			(at 161.925 43.18 0)
 			(hide yes)
@@
 			)
 		)
-		(property "Digi-Key PN" ""
+		(property "Digi-Key PN" "311-100KLRCT-ND"
 			(at 69.85 30.48 0)
 			(hide yes)
@@
 			)
 		)
-		(property "Digi-Key PN" ""
+		(property "Digi-Key PN" "311-100KLRCT-ND"
 			(at 190.5 30.48 0)
 			(hide yes)
@@
 			)
 		)
-		(property "Digi-Key PN" ""
+		(property "Digi-Key PN" "1276-CL05B104KB5NNNCCT-ND"
 			(at 104.775 152.4 0)
 			(hide yes)
@@
 			)
 		)
-		(property "Ampacity" "0.7A"
+		(property "Ampacity" "1.3A"
 			(at 204.47 83.82 90)
 			(show_name no)
@@
 			)
 		)
+		(property "Digi-Key PN" "490-16508-1-ND"
+			(at 204.47 90.17 0)
+			(hide yes)
+			(show_name no)
+			(do_not_autoplace no)
+			(effects
+				(font
+					(size 1.27 1.27)
+				)
+			)
+		)
 		(pin "2"
 		)
@@
 			)
 		)
-		(property "Digi-Key PN" ""
+		(property "Digi-Key PN" "311-1.00KLRCT-ND"
 			(at 41.91 92.71 0)
 			(hide yes)
@@
 			)
 		)
-		(property "Digi-Key PN" ""
+		(property "Digi-Key PN" "YAG3503CT-ND"
 			(at 208.28 114.3 0)
 			(hide yes)
@@
 	)
 	(symbol
-		(lib_id "Logic_LevelTranslator:TXB0102YZP")
+		(lib_id "Logic_LevelTranslator:TXB0102DCU")
 		(at 130.81 39.37 0)
 		(mirror y)
@@
 			)
 		)
-		(property "Value" "TXB0102YZP"
+		(property "Value" "TXB0102DCU"
 			(at 127 27.94 0)
 			(show_name no)
@@
 			)
 		)
-		(property "Footprint" "Package_BGA:Texas_DSBGA-8_0.9x1.9mm_Layout2x4_P0.5mm"
+		(property "Footprint" "Package_SO:VSSOP-8_2.3x2mm_P0.5mm"
 			(at 130.81 53.34 0)
 			(hide yes)
@@
 			)
 		)
-		(property "Description" "2-Bit Bidirectional Voltage-Level Translator With Auto Direction Sensing and ±15-kV ESD Protection, DSBGA-8"
+		(property "Description" "2-Bit Bidirectional Voltage-Level Translator With Auto Direction Sensing and ±15-kV ESD Protection, VSSOP-8"
 			(at 130.81 39.37 0)
 			(hide yes)
@@
 			)
 		)
-		(pin "B2"
+		(property "Digi-Key PN" "296-22862-1-ND"
+			(at 130.81 39.37 0)
+			(hide yes)
+			(show_name no)
+			(do_not_autoplace no)
+			(effects
+				(font
+					(size 1.27 1.27)
+				)
+			)
+		)
+		(pin "7"
 		)
-		(pin "D2"
+		(pin "5"
 		)
-		(pin "C2"
+		(pin "6"
 		)
-		(pin "B1"
+		(pin "2"
 		)
-		(pin "A2"
+		(pin "8"
 		)
-		(pin "D1"
+		(pin "4"
 		)
-		(pin "A1"
+		(pin "1"
 		)
-		(pin "C1"
+		(pin "3"
 		)
 		(instances
@@
 			)
 		)
-		(property "Digi-Key PN" ""
+		(property "Digi-Key PN" "311-1.00KLRCT-ND"
 			(at 29.21 92.71 0)
 			(hide yes)
@@
 			)
 		)
-		(property "Digi-Key PN" ""
+		(property "Digi-Key PN" "1276-CL05A106MP6NUN8CT-ND"
 			(at 113.03 55.88 0)
 			(hide yes)
@@
 			)
 		)
-		(property "Digi-Key PN" ""
+		(property "Digi-Key PN" "YAG3503CT-ND"
 			(at 111.76 166.37 0)
 			(hide yes)
@@
 			)
 		)
-		(property "Ampacity" "0.7A"
+		(property "Ampacity" "1.3A"
 			(at 248.92 138.4299 0)
 			(show_name no)
@@
 			)
 		)
+		(property "Digi-Key PN" "490-16508-1-ND"
+			(at 247.65 134.62 0)
+			(hide yes)
+			(show_name no)
+			(do_not_autoplace no)
+			(effects
+				(font
+					(size 1.27 1.27)
+				)
+			)
+		)
 		(pin "2"
 		)
@@
 			)
 		)
-		(property "Digi-Key PN" ""
+		(property "Digi-Key PN" "1276-CL05A106MP6NUN8CT-ND"
 			(at 45.72 152.4 0)
 			(hide yes)
@@
 			)
 		)
-		(property "Digi-Key PN" ""
+		(property "Digi-Key PN" "1276-CL05A106MP6NUN8CT-ND"
 			(at 66.04 152.4 0)
 			(hide yes)
@@
 			)
 		)
-		(property "Digi-Key PN" ""
+		(property "Digi-Key PN" "732-11992-1-ND"
 			(at 292.608 307.594 0)
 			(hide yes)

Commit message: update some design notes
Other:
- note added: "Datasheet gives conflicting rules Says VCCB > VCCA, but says outputs go HiZ when either supply is not up"
Changed lines of the file:
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@@
+		)
+	)
+	(text "Datasheet gives conflicting rules\nSays VCCB > VCCA, but says outputs go HiZ\nwhen either supply is not up"
+		(exclude_from_sim no)
+		(at 77.47 16.51 0)
+		(effects
+			(font
+				(size 1.27 1.27)
+			)
+			(justify left)
 		)
 	)

Commit message: add new digikey pns
Parts:
- R905, R909, R910: Digi-Key PN YAG3503CT-ND -> 311-5.10KLRCT-ND
Changed lines of the file:
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@@
 			)
 		)
-		(property "Digi-Key PN" "YAG3503CT-ND"
+		(property "Digi-Key PN" "311-5.10KLRCT-ND"
 			(at 195.58 114.3 0)
 			(hide yes)
@@
 			)
 		)
-		(property "Digi-Key PN" "YAG3503CT-ND"
+		(property "Digi-Key PN" "311-5.10KLRCT-ND"
 			(at 208.28 114.3 0)
 			(hide yes)
@@
 			)
 		)
-		(property "Digi-Key PN" "YAG3503CT-ND"
+		(property "Digi-Key PN" "311-5.10KLRCT-ND"
 			(at 111.76 166.37 0)
 			(hide yes)
