File: hdw/DSP_board/rev_a/Audio_Visualiser_DSP/Audio_Visualiser_DSP.kicad_pcb (KiCad board)
At the start: 2 copper layers, 100 x 50 mm, 388 parts, among them J1001 I2C, J1002 UART, J1004 LED SPI, J1301 Switchcraft_PJRAN2X1U_X, J1302 RCA Left TP, J1303 RCA Right TP, J1401 Left, J1402 Right, J1403 Speaker Left TP, J1404 Speaker Right TP, J1501 Gain Left TP, J1502 Gain Right TP, J1503 Mux Left TP, J1504 Mux Right TP, J1601 ADC Left TP, J1602 ADC Right TP, J1901 Power, J1902 Power, J1903 Conn_01x06, J201 +12V IN, J2101 Left, J2102 Right, J601 PICKIT4, J801 Boot Audio Source Select, J901 USB_C_Receptacle_USB2.0_14P, Q401 BSS214NW, Q402 BSS214NW, Q601 BSS214NW, SW1901 Cap_Touch, SW1902 Power, SW601 MRST, U1001 DS1683, U1002 MCP9804, U1101 74LVC1G97, U1102 74LVC1G97, U1103 74LVC1G97, U1104 74LVC1G97, U1105 74LVC1G97, U1106 74LVC1G97, U1201 74LVC1G97, U1202 74LVC1G97, U1203 74LVC1G97, U1301 MCP6N11-001, U1302 MCP6N11-001, U1401 MCP6N11-001, U1402 MCP6N11-001, U1501 TS3A24159DRC, U1502 MCP6024, U1503 MCP4451-103E/ML, U1601 MCP6024, U1701 MCP6024, U1702 REF35160QDBVR, U1801 74LVC1G97, U1802 74LVC1G97, U1803 74VHC541BQ,115, U1804 74VHC541BQ,115, U1805 74LVC1G97, U1806 74LVC1G97, U1807 TCA9801, U1808 74LVC1G97, U1809 TCA9801, U1901 AT42QT1010-TSHR, U1902 74LVC1G97, U1903 74LVC1G97, U201 TPS259474LRPWR, U301 INA231A, U302 MCP9804, U401 74LVC1G97, U402 TPS62150A, U501 INA231A, U502 MCP9804, U601 74LVC1G97, U701 dsPIC33AK256MPS105, U801 PCA9536DP, U802 74LVC1G97, U803 TCA9801, U805 74LVC1G97, U901 CP2104, U902 74LVC1G97, U903 TXB0102DCU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

Commit message: more component placement
Parts:
- C701, C704, C706, C707, C708, C711, C714, C716, C801, C802, C803, C804, C805, R801, R807: moved to B.Cu
- moved R801 435.2 mm to (497.8, 131.8)
- moved C802 432.3 mm to (497.8, 132.8)
- moved R807 429.2 mm to (492.0, 141.7), turned to 180 degrees
- moved C804 427.5 mm to (493.3, 131.3), turned to -90 degrees
- moved C805 426.6 mm to (492.0, 140.7), turned to 180 degrees
- moved C803 426.5 mm to (492.3, 131.3), turned to -90 degrees
- moved R802 425.1 mm to (487.9, 130.8)
- moved R804 425.0 mm to (487.9, 131.8)
- moved U802 419.8 mm to (497.8, 132.8), turned to 180 degrees
- moved U803 417.4 mm to (492.8, 131.3)
- moved J801 415.0 mm to (484.1, 136.9)
- moved U805 414.2 mm to (492.0, 140.7)
- moved C801 413.0 mm to (478.0, 139.4), turned to 180 degrees
- moved R803 411.2 mm to (473.7, 138.4), turned to 180 degrees
- moved R805 411.0 mm to (473.7, 139.4), turned to 180 degrees
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Other:
- board text added: "DSP"
- board text added: "DSP MISC"
- board text added: "USB"

Commit message: place some more components
Parts:
- removed FB603: 220, project_lib:L_0402
- added R610: 10, project_lib:R_0402, B.Cu at (535.9, 108.6)
- C1201, C601, C604, C605, D601, R1201, R1203, R602, R604, R605, R607, R608: moved to B.Cu
- moved C604 412.1 mm to (537.5, 108.6), turned to -90 degrees
- moved C605 399.9 mm to (538.0, 102.2), turned to -90 degrees
- moved C603 399.2 mm to (537.5, 106.3)
- moved R606 397.2 mm to (540.8, 108.6), turned to -90 degrees
- moved R601 396.9 mm to (538.0, 112.4)
- moved C601 396.1 mm to (534.2, 97.4), turned to 180 degrees
- moved Q601 395.5 mm to (536.7, 102.2)
- moved R605 395.3 mm to (539.0, 108.6), turned to -90 degrees
- moved J601 394.4 mm to (519.2, 94.3), turned to 180 degrees
- moved R603 394.0 mm to (534.7, 102.2), turned to 90 degrees
- moved R602 393.6 mm to (534.2, 98.4), turned to 180 degrees
- moved R609 393.0 mm to (539.0, 102.2), turned to 90 degrees
- moved R608 392.9 mm to (539.0, 102.2), turned to 90 degrees
- moved U601 392.7 mm to (534.2, 97.4)
- moved R604 392.4 mm to (535.9, 102.2), turned to -90 degrees
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
Commit message: arranged LEDs
Parts:
- C1101, C1102, C1103, C1104, C1105, C1106, C1202, C1203, R1101, R1102, R1103, R1104, R1105, R1106, R1107, R1202, R1204, R1205, R1206: moved to B.Cu
- moved R1107 232.4 mm to (323.9, 192.0), turned to 90 degrees
- moved U1106 232.3 mm to (321.6, 192.0)
- moved U1105 232.2 mm to (321.6, 188.0)
- moved U1104 232.1 mm to (321.6, 183.9)
- moved R1106 232.0 mm to (323.9, 188.0), turned to 90 degrees
- moved U1103 232.0 mm to (321.6, 179.8)
- moved U1102 231.9 mm to (321.6, 175.8)
- moved U1101 231.8 mm to (321.6, 171.7)
- moved R1105 231.6 mm to (323.9, 183.9), turned to 90 degrees
- moved R1104 231.3 mm to (323.9, 179.8), turned to 90 degrees
- moved R1103 230.9 mm to (323.9, 175.8), turned to 90 degrees
- moved R1102 230.5 mm to (323.9, 171.7), turned to 90 degrees
- moved R1101 228.9 mm to (321.6, 172.7)
- moved C1106 228.1 mm to (321.6, 192.0), turned to 180 degrees
- moved C1105 227.6 mm to (321.6, 188.0), turned to 180 degrees
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Other:
- board text added: "+12V"
- board text added: "+3.3V"
- board text added: "ERROR"
- board text added: "HRTBT"
- board text added: "LEDs"
- board text added: "Left LED +3.3V"
- board text added: "Left VLED"
- board text added: "RESET"
- board text added: "Right LED +3.3V"
- board text added: "Right VLED"

Commit message: much more component placement
Parts:
- removed J1902: Power, project_lib:TerminalBlock_Phoenix_MKDS-1,5-2-5.08_1x02_P5.08mm_Horizontal
- added R1910: 0, project_lib:R_0402, B.Cu at (386.1, 174.5)
- C1301, C1302, C1303, C1304, C1305, C1306, C1401, C1402, C1403, C1404, C1901, C1902, C1903, C1904, C1905, C1906, C2101, D1301, D1302, D1303, D1304, D1305, D1306, D1307, D1308, D1309, D1310, D1311, D1312, D1401, D1402, D1403, D1404, D1405, D1406, D1407, D1408, D2101, D2103, R1309, R1310, R1311, R1312, R1313, R1314, R1405, R1406, R1407, R1408, R1902, R1903, R1905, R1907, R1909: moved to B.Cu
- moved R1303 480.6 mm to (599.9, 136.4), turned to 90 degrees
- moved R1308 477.9 mm to (599.1, 139.2), turned to 90 degrees
- moved R1304 477.8 mm to (597.4, 136.4), turned to 90 degrees
- moved R1307 477.2 mm to (598.0, 139.2), turned to 90 degrees
- moved R1310 476.8 mm to (598.0, 143.2), turned to -90 degrees
- moved R1314 475.9 mm to (599.1, 143.2), turned to -90 degrees
- moved R1312 475.6 mm to (599.7, 127.0), turned to -90 degrees
- moved J1301 475.3 mm to (598.9, 124.0), turned to 180 degrees
- moved R1317 475.1 mm to (598.5, 147.8), turned to -90 degrees
- moved R1318 473.7 mm to (597.5, 147.8), turned to 90 degrees
- moved D1303 471.6 mm to (599.9, 136.4), turned to 90 degrees
- moved D1304 468.7 mm to (597.4, 136.4), turned to 90 degrees
- moved R1301 466.5 mm to (585.0, 136.4), turned to 90 degrees
- moved D1307 465.0 mm to (596.8, 141.2)
- moved R1306 464.6 mm to (584.3, 139.2), turned to 90 degrees
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Connections:
- J1901 pad 2: Net-(J1901-Pin_1) -> GND
Other:
- board text added: "Buttons"
- board text added: "RCA Amps"
- board text added: "Speaker amps"

Commit message: expanded board edge, placed mount holes and IO connectors
Parts:
- C2102, D2102, D2104: moved to B.Cu
- moved D2103 370.6 mm to (98.9, 136.7), turned to 180 degrees
- moved D2102 362.3 mm to (160.3, 136.6), turned to 180 degrees
- moved D2104 358.4 mm to (147.9, 136.7), turned to 180 degrees
- moved D2101 354.6 mm to (111.4, 136.6), turned to 180 degrees
- moved C2101 341.5 mm to (121.8, 136.7), turned to 180 degrees
- moved J2101 340.3 mm to (125.6, 142.0), turned to -90 degrees
- moved C2102 339.0 mm to (170.7, 136.7), turned to 180 degrees
- moved J2102 321.2 mm to (174.6, 142.0), turned to -90 degrees
- moved H2004 102.4 mm to (86.3, 132.4)
- moved H2001 77.6 mm to (86.3, 53.1)
- moved H2003 76.8 mm to (178.3, 132.4)
- moved H2002 15.6 mm to (178.3, 53.1)
Connections:
- D2101 pad 1: LEFT_LED_DRIVER_SPI_SDO_BUF -> LEFT_LED_DRIVER_SPI_SCK_BUF
- D2101 pad 3: LEFT_LED_DRIVER_SPI_SCK_BUF -> LEFT_LED_DRIVER_SPI_SDO_BUF
- D2101 pad 4: LEFT_VLED_RUN_BUF -> LEFT_LED_DRIVER_BLANK_PWM_BUF
- D2101 pad 6: LEFT_LED_DRIVER_BLANK_PWM_BUF -> LEFT_VLED_RUN_BUF
- D2102 pad 1: RIGHT_LED_DRIVER_SPI_SDO_BUF -> RIGHT_LED_DRIVER_SPI_SCK_BUF
- D2102 pad 3: RIGHT_LED_DRIVER_SPI_SCK_BUF -> RIGHT_LED_DRIVER_SPI_SDO_BUF
- D2102 pad 4: RIGHT_VLED_RUN_BUF -> RIGHT_LED_DRIVER_BLANK_PWM_BUF
- D2102 pad 6: RIGHT_LED_DRIVER_BLANK_PWM_BUF -> RIGHT_VLED_RUN_BUF
- D2103 pad 1: LEFT_LED_POS3P3_PGOOD_BUF -> LEFT_LED_POS3P3_RUN_BUF
- D2103 pad 3: LEFT_LED_POS3P3_RUN_BUF -> LEFT_LED_POS3P3_PGOOD_BUF
- D2103 pad 4: LEFT_I2C_SDA -> LEFT_VLED_PGOOD_BUF
- D2103 pad 6: LEFT_VLED_PGOOD_BUF -> LEFT_I2C_SDA
- D2104 pad 1: RIGHT_LED_POS3P3_PGOOD_BUF -> RIGHT_LED_POS3P3_RUN_BUF
- D2104 pad 3: RIGHT_LED_POS3P3_RUN_BUF -> RIGHT_LED_POS3P3_PGOOD_BUF
- D2104 pad 4: RIGHT_I2C_SDA -> RIGHT_VLED_PGOOD_BUF
- D2104 pad 6: RIGHT_VLED_PGOOD_BUF -> RIGHT_I2C_SDA
Other:
- board size 100 x 50 mm -> 100 x 100 mm

Commit message: Starting placing higher level blocks within board outline
Parts:
- C1303, C1304, C1305, C1306, C1401, C1402, C1403, C1404, D1305, D1306, D1307, D1308, D1309, D1310, D1311, D1312, D1401, D1402, D1403, D1404, D1405, D1406, D1407, D1408, R1309, R1310, R1313, R1314, R1405, R1406, R1407, R1408: moved to F.Cu
- D201, R1305, R1306, R1307, R1308, R1315, R1316, R1317, R1318, R1401, R1402, R1403, R1404, R1409, R1410, R1411, R1412, U1301, U1302, U1401, U1402: moved to B.Cu
- moved D1311 439.8 mm to (166.1, 71.3), turned to 0 degrees
- moved D1312 439.8 mm to (166.1, 69.3), turned to 180 degrees
- moved D1309 439.8 mm to (151.4, 71.3), turned to 0 degrees
- moved D1310 439.8 mm to (151.4, 69.3), turned to 180 degrees
- moved C1305 439.3 mm to (151.6, 76.4)
- moved C1306 438.7 mm to (166.7, 76.4)
- moved R1306 437.3 mm to (152.6, 69.3)
- moved R1308 437.3 mm to (167.4, 69.3)
- moved R1314 437.3 mm to (167.4, 73.3)
- moved C1303 437.3 mm to (152.6, 76.4)
- moved R1313 437.3 mm to (152.6, 73.3)
- moved C1304 436.8 mm to (167.6, 76.4)
- moved R1315 436.8 mm to (152.9, 77.9)
- moved U1301 436.6 mm to (153.0, 74.9)
- moved D1302 436.3 mm to (151.7, 66.5)
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Other:
- board text removed: "Input Power"
- board text removed: "Panel Buffers"
- board text removed: "RCA Amps"
