File: hdw/DSP_board/rev_a/Audio_Visualiser_DSP/pinout_fix_backup_20261001_174045/dspic33_power.kicad_sch (KiCad schematic)
At the start: 21 parts, among them U701 dsPIC33AK256MPS105

Commit message: fixed dsPIC pinout to add exposed pad, fixed footprint mapping. Fixed +12V connection to INA
Parts:
- U701: footprint Package_DFN_QFN:VQFN-48-1EP_6x6mm_P0.4mm_EP4.1x4.1mm -> Package_DFN_QFN:QFN-48-1EP_6x6mm_P0.4mm_EP4.1x4.1mm
Connections:
- net GND: no longer U701.49 (VSS)
Changed lines of the file:
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@@
 			)
 		)
-		(property "Footprint" "Package_DFN_QFN:VQFN-48-1EP_6x6mm_P0.4mm_EP4.1x4.1mm"
+		(property "Footprint" "Package_DFN_QFN:QFN-48-1EP_6x6mm_P0.4mm_EP4.1x4.1mm"
 			(at 137.16 52.07 0)
 			(hide yes)
@@
 		(pin "39"
 		)
-		(pin "49"
-		)
 		(instances
