File: hdw/DSP_board/rev_a/Audio_Visualiser_DSP/pn_assign_backup_20261008_193815/POS3P3_power_supply.kicad_sch (KiCad schematic)
At the start: 25 parts, among them Q401 BSS214NW, Q402 ZXMS6004FFTA, U401 74LVC1G97, U402 TPS62150A

Commit message: add new digikey pns
Parts:
- C402, C403: Digi-Key PN 445-6862-1-ND -> 1276-1075-1-ND
- C406, C407, C408: Digi-Key PN 478-KGM21AR71A106KUCT-ND -> 490-14381-1-ND
- D401: value BAT43WS -> BAT54J; Digi-Key PN BAT43WSRRGCT-ND -> (none)
- R409: Digi-Key PN YAG3146CT-ND -> 311-3.16KLRCT-ND
Changed lines of the file:
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@@
 			)
 		)
-		(property "Digi-Key PN" "478-KGM21AR71A106KUCT-ND"
+		(property "Digi-Key PN" "490-14381-1-ND"
 			(at 210.185 123.19 0)
 			(hide yes)
@@
 			)
 		)
-		(property "Digi-Key PN" "478-KGM21AR71A106KUCT-ND"
+		(property "Digi-Key PN" "490-14381-1-ND"
 			(at 200.025 44.45 0)
 			(hide yes)
@@
 			)
 		)
-		(property "Digi-Key PN" "YAG3146CT-ND"
+		(property "Digi-Key PN" "311-3.16KLRCT-ND"
 			(at 222.25 69.85 0)
 			(hide yes)
@@
 			)
 		)
-		(property "Digi-Key PN" "478-KGM21AR71A106KUCT-ND"
+		(property "Digi-Key PN" "490-14381-1-ND"
 			(at 184.785 44.45 0)
 			(hide yes)
@@
 			)
 		)
-		(property "Digi-Key PN" "445-6862-1-ND"
+		(property "Digi-Key PN" "1276-1075-1-ND"
 			(at 100.965 36.83 0)
 			(hide yes)
@@
 			)
 		)
-		(property "Digi-Key PN" "445-6862-1-ND"
+		(property "Digi-Key PN" "1276-1075-1-ND"
 			(at 81.915 36.83 0)
 			(hide yes)
@@
 			)
 		)
-		(property "Value" "BAT43WS"
+		(property "Value" "BAT54J"
 			(at 201.93 123.5076 90)
 			(show_name no)
@@
 			(at 199.39 124.46 0)
 			(hide yes)
-			(show_name no)
-			(do_not_autoplace no)
-			(effects
-				(font
-					(size 1.27 1.27)
-				)
-			)
-		)
-		(property "Digi-Key PN" "BAT43WSRRGCT-ND"
-			(at 199.39 124.46 0)
-			(hide yes)
