File: hdw/DSP_board/rev_a/Audio_Visualiser_DSP/pn_assign_backup_20261008_193815/anti_alias_filtering.kicad_sch (KiCad schematic)
At the start: 21 parts, among them J1601 ADC Left TP, J1602 ADC Right TP, U1601 MCP6024

Commit message: add new digikey pns
Parts:
- C1606: Digi-Key PN 490-18202-1-ND -> 445-9116-1-ND
Changed lines of the file:
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@@
 			)
 		)
-		(property "Digi-Key PN" "490-18202-1-ND"
+		(property "Digi-Key PN" "445-9116-1-ND"
 			(at 144.145 21.59 0)
 			(hide yes)
