File: hdw/DSP_board/rev_a/Audio_Visualiser_DSP/pn_assign_backup_20261008_193815/audio_voltage_references.kicad_sch (KiCad schematic)
At the start: 11 parts, among them U1701 MCP6024, U1702 REF35160QDBVR

Commit message: add new digikey pns
Parts:
- C1703, C1705: Digi-Key PN 490-18202-1-ND -> 445-9116-1-ND
Changed lines of the file:
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@@
 			)
 		)
-		(property "Digi-Key PN" "490-18202-1-ND"
+		(property "Digi-Key PN" "445-9116-1-ND"
 			(at 149.225 26.67 0)
 			(hide yes)
@@
 			)
 		)
-		(property "Digi-Key PN" "490-18202-1-ND"
+		(property "Digi-Key PN" "445-9116-1-ND"
 			(at 98.425 86.36 0)
 			(hide yes)
