File: hdw/DSP_board/rev_a/Audio_Visualiser_DSP/pn_assign_backup_20261008_193815/dspic33_gpio.kicad_sch (KiCad schematic)
At the start: 20 parts, among them J801 Boot Audio Source Select, U801 PCA9536DP, U802 74LVC1G97, U803 TCA9803, U804 dsPIC33AK256MPS105, U805 74LVC1G97

Commit message: add new digikey pns
Parts:
- H801: Digi-Key PN S9337-ND -> QPC02SXGN-RC
- U805: Digi-Key PN 296-15582-1-ND -> (none)
Changed lines of the file:
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@@
 			)
 		)
-		(property "Digi-Key PN" "S9337-ND"
+		(property "Digi-Key PN" "QPC02SXGN-RC"
 			(at 138.43 20.32 0)
 			(hide yes)
@@
 			(at 204.47 27.94 0)
 			(hide yes)
-			(show_name no)
-			(do_not_autoplace no)
-			(effects
-				(font
-					(size 1.27 1.27)
-				)
-			)
-		)
-		(property "Digi-Key PN" "296-15582-1-ND"
-			(at 204.47 27.94 0)
-			(hide yes)
