File: hdw/DSP_board/rev_a/Audio_Visualiser_DSP/pn_assign_backup_20261008_193815/led_panel_connectors.kicad_sch (KiCad schematic)
At the start: 8 parts, among them J2101 Left, J2102 Right

Commit message: add new digikey pns
Parts:
- C2101, C2102: Digi-Key PN 445-6862-1-ND -> 1276-1075-1-ND
Changed lines of the file:
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@@
 			)
 		)
-		(property "Digi-Key PN" "445-6862-1-ND"
+		(property "Digi-Key PN" "1276-1075-1-ND"
 			(at 234.315 30.48 0)
 			(hide yes)
@@
 			)
 		)
-		(property "Digi-Key PN" "445-6862-1-ND"
+		(property "Digi-Key PN" "1276-1075-1-ND"
 			(at 234.315 96.52 0)
 			(hide yes)
