File: hdw/DSP_board/rev_a/Audio_Visualiser_DSP/pn_assign_backup_20261008_193815/platform_etc.kicad_sch (KiCad schematic)
At the start: 14 parts, among them J1001 I2C, J1002 UART, J1003 AUDIO, J1004 LED SPI, U1001 DS1683, U1002 MCP9804

Commit message: add new digikey pns
Parts:
- D1001: value BAT43WS -> BAT54J; Digi-Key PN BAT43WSRRGCT-ND -> (none)
Changed lines of the file:
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@@
 			)
 		)
-		(property "Value" "BAT43WS"
+		(property "Value" "BAT54J"
 			(at 60.96 34.6074 90)
 			(show_name no)
@@
 			)
 		)
-		(property "Digi-Key PN" "BAT43WSRRGCT-ND"
-			(at 58.42 34.29 0)
-			(hide yes)
-			(show_name no)
-			(do_not_autoplace no)
-			(effects
-				(font
-					(size 1.27 1.27)
-				)
-			)
-		)
