File: hdw/DSP_board/rev_a/Audio_Visualiser_DSP/pn_assign_backup_20261008_193815/pushbuttons.kicad_sch (KiCad schematic)
At the start: 25 parts, among them J1901 Power, J1902 Power, J1903 Conn_01x06, SW1901 Cap_Touch, SW1902 Power, U1901 AT42QT1010-TSHR, U1902 74LVC1G97, U1903 74LVC1G97

Commit message: add new digikey pns
Parts:
- C1902, C1906: Digi-Key PN 445-5942-1-ND -> 490-11917-1-ND
- C1903: Digi-Key PN 490-18202-1-ND -> 445-9116-1-ND
- J1903: Digi-Key PN 35-PRPC003DAAN-RC-ND -> PRPC003DAAN-RC
Changed lines of the file:
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@@
 			)
 		)
-		(property "Digi-Key PN" "490-18202-1-ND"
+		(property "Digi-Key PN" "445-9116-1-ND"
 			(at 83.185 74.93 0)
 			(hide yes)
@@
 			)
 		)
-		(property "Digi-Key PN" "35-PRPC003DAAN-RC-ND"
+		(property "Digi-Key PN" "PRPC003DAAN-RC"
 			(at 116.84 142.24 0)
 			(hide yes)
@@
 			)
 		)
-		(property "Digi-Key PN" "445-5942-1-ND"
+		(property "Digi-Key PN" "490-11917-1-ND"
 			(at 145.415 43.18 0)
 			(hide yes)
@@
 			)
 		)
-		(property "Digi-Key PN" "445-5942-1-ND"
+		(property "Digi-Key PN" "490-11917-1-ND"
 			(at 74.295 44.45 0)
 			(hide yes)
