File: hdw/DSP_board/rev_a/Audio_Visualiser_DSP/pn_assign_backup_20261008_193815/rca_signal_conditioning.kicad_sch (KiCad schematic)
At the start: 41 parts, among them J1301 Switchcraft_PJRAN2X1U_X, J1302 RCA Left TP, J1303 RCA Right TP, U1301 MCP6N11-001, U1302 MCP6N11-001

Commit message: add new digikey pns
Parts:
- C1305, C1306: Digi-Key PN 490-18202-1-ND -> 445-9116-1-ND
- D1305, D1306, D1307, D1308, D1309, D1310, D1311, D1312: value BAT43WS -> BAT54J; Digi-Key PN BAT43WSRRGCT-ND -> (none)
- R1305, R1306, R1307, R1308: Digi-Key PN 311-30.0KLRCT-ND -> (none)
- R1311, R1312: Digi-Key PN 311-10.0LRCT-ND -> (none)
- U1301, U1302: Digi-Key PN MCP6N11T-001E/MNYCT-ND -> (none)
Changed lines of the file:
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@@
 			)
 		)
-		(property "Digi-Key PN" "311-30.0KLRCT-ND"
+		(property "Digi-Key PN" ""
 			(at 102.87 60.96 0)
 			(hide yes)
@@
 			)
 		)
-		(property "Digi-Key PN" "311-10.0LRCT-ND"
+		(property "Digi-Key PN" ""
 			(at 113.03 163.83 0)
 			(hide yes)
@@
 			)
 		)
-		(property "Digi-Key PN" "490-18202-1-ND"
+		(property "Digi-Key PN" "445-9116-1-ND"
 			(at 175.895 12.7 0)
 			(hide yes)
@@
 			)
 		)
-		(property "Digi-Key PN" "MCP6N11T-001E/MNYCT-ND"
-			(at 179.07 118.11 0)
-			(hide yes)
-			(show_name no)
-			(do_not_autoplace no)
-			(effects
-				(font
-					(size 1.27 1.27)
-				)
-			)
-		)
 		(pin "6"
 		)
@@
 			)
 		)
-		(property "Value" "BAT43WS"
+		(property "Value" "BAT54J"
 			(at 138.43 126.6824 90)
 			(show_name no)
@@
 			)
 		)
-		(property "Digi-Key PN" "BAT43WSRRGCT-ND"
-			(at 135.89 125.73 0)
-			(hide yes)
-			(show_name no)
-			(do_not_autoplace no)
-			(effects
-				(font
-					(size 1.27 1.27)
-				)
-			)
-		)
 		(pin "2"
 		)
@@
 			)
 		)
-		(property "Value" "BAT43WS"
+		(property "Value" "BAT54J"
 			(at 156.21 47.9424 90)
 			(show_name no)
@@
 			)
 		)
-		(property "Digi-Key PN" "BAT43WSRRGCT-ND"
-			(at 153.67 46.99 0)
-			(hide yes)
-			(show_name no)
-			(do_not_autoplace no)
-			(effects
-				(font
-					(size 1.27 1.27)
-				)
-			)
-		)
 		(pin "2"
 		)
@@
 			)
 		)
-		(property "Digi-Key PN" "311-30.0KLRCT-ND"
+		(property "Digi-Key PN" ""
 			(at 102.87 124.46 0)
 			(hide yes)
@@
 			)
 		)
-		(property "Value" "BAT43WS"
+		(property "Value" "BAT54J"
 			(at 138.43 63.1824 90)
 			(show_name no)
@@
 			)
 		)
-		(property "Digi-Key PN" "BAT43WSRRGCT-ND"
-			(at 135.89 62.23 0)
-			(hide yes)
-			(show_name no)
-			(do_not_autoplace no)
-			(effects
-				(font
-					(size 1.27 1.27)
-				)
-			)
-		)
 		(pin "2"
 		)
@@
 			)
 		)
-		(property "Digi-Key PN" "490-18202-1-ND"
+		(property "Digi-Key PN" "445-9116-1-ND"
 			(at 175.895 76.2 0)
 			(hide yes)
@@
 			)
 		)
-		(property "Value" "BAT43WS"
+		(property "Value" "BAT54J"
 			(at 156.21 111.4424 90)
 			(show_name no)
@@
 			)
 		)
-		(property "Digi-Key PN" "BAT43WSRRGCT-ND"
-			(at 153.67 110.49 0)
-			(hide yes)
-			(show_name no)
-			(do_not_autoplace no)
-			(effects
-				(font
-					(size 1.27 1.27)
-				)
-			)
-		)
 		(pin "2"
 		)
@@
 			)
 		)
-		(property "Value" "BAT43WS"
+		(property "Value" "BAT54J"
 			(at 138.43 47.9424 90)
 			(show_name no)
@@
 			)
 		)
-		(property "Digi-Key PN" "BAT43WSRRGCT-ND"
-			(at 135.89 46.99 0)
-			(hide yes)
-			(show_name no)
-			(do_not_autoplace no)
-			(effects
-				(font
-					(size 1.27 1.27)
-				)
-			)
-		)
 		(pin "2"
 		)
@@
 			)
 		)
-		(property "Value" "BAT43WS"
+		(property "Value" "BAT54J"
 			(at 156.21 126.6824 90)
 			(show_name no)
@@
 			)
 		)
-		(property "Digi-Key PN" "BAT43WSRRGCT-ND"
-			(at 153.67 125.73 0)
-			(hide yes)
-			(show_name no)
-			(do_not_autoplace no)
-			(effects
-				(font
-					(size 1.27 1.27)
-				)
-			)
-		)
 		(pin "2"
 		)
@@
 			)
 		)
-		(property "Digi-Key PN" "311-30.0KLRCT-ND"
+		(property "Digi-Key PN" ""
 			(at 102.87 63.5 0)
 			(hide yes)
@@
 			)
 		)
-		(property "Digi-Key PN" "311-30.0KLRCT-ND"
+		(property "Digi-Key PN" ""
 			(at 102.87 127 0)
 			(hide yes)
@@
 			)
 		)
-		(property "Digi-Key PN" "311-10.0LRCT-ND"
+		(property "Digi-Key PN" ""
 			(at 113.03 181.61 0)
 			(hide yes)
@@
 			)
 		)
-		(property "Value" "BAT43WS"
+		(property "Value" "BAT54J"
 			(at 138.43 111.4424 90)
 			(show_name no)
@@
 			)
 		)
-		(property "Digi-Key PN" "BAT43WSRRGCT-ND"
-			(at 135.89 110.49 0)
-			(hide yes)
-			(show_name no)
-			(do_not_autoplace no)
-			(effects
-				(font
-					(size 1.27 1.27)
-				)
-			)
-		)
 		(pin "2"
 		)
@@
 			)
 		)
-		(property "Digi-Key PN" "MCP6N11T-001E/MNYCT-ND"
-			(at 179.07 54.61 0)
-			(hide yes)
-			(show_name no)
-			(do_not_autoplace no)
-			(effects
-				(font
-					(size 1.27 1.27)
-				)
-			)
-		)
 		(pin "6"
 		)
@@
 			)
 		)
-		(property "Value" "BAT43WS"
+		(property "Value" "BAT54J"
 			(at 156.21 63.1824 90)
 			(show_name no)
@@
 			(at 153.67 62.23 0)
 			(hide yes)
-			(show_name no)
-			(do_not_autoplace no)
-			(effects
-				(font
-					(size 1.27 1.27)
-				)
-			)
-		)
-		(property "Digi-Key PN" "BAT43WSRRGCT-ND"
-			(at 153.67 62.23 0)
-			(hide yes)
