File: hdw/DSP_board/rev_a/Audio_Visualiser_DSP/pn_assign_backup_20261008_193815/source_selection_pgas.kicad_sch (KiCad schematic)
At the start: 17 parts, among them J1501 Gain Left TP, J1502 Gain Right TP, J1503 Mux Left TP, J1504 Mux Right TP, U1501 TS3A24159DRC, U1502 MCP6024, U1503 MCP4451-103E/ML

Commit message: add new digikey pns
Parts:
- C1502, C1504, C1506: Digi-Key PN 490-18202-1-ND -> 445-9116-1-ND
Changed lines of the file:
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@@
 			)
 		)
-		(property "Digi-Key PN" "490-18202-1-ND"
+		(property "Digi-Key PN" "445-9116-1-ND"
 			(at 142.875 19.05 0)
 			(hide yes)
@@
 			)
 		)
-		(property "Digi-Key PN" "490-18202-1-ND"
+		(property "Digi-Key PN" "445-9116-1-ND"
 			(at 244.475 125.73 0)
 			(hide yes)
@@
 			)
 		)
-		(property "Digi-Key PN" "490-18202-1-ND"
+		(property "Digi-Key PN" "445-9116-1-ND"
 			(at 36.195 119.38 0)
 			(hide yes)
