File: hdw/DSP_board/rev_a/Audio_Visualiser_DSP/pn_assign_backup_20261008_193815/usb_uart_bridge.kicad_sch (KiCad schematic)
At the start: 32 parts, among them J901 USB_C_Receptacle_USB2.0_14P, U901 CP2104, U902 74LVC1G97, U903 TXB0102DCU, U904 TPD3S014DBVR

Commit message: add new digikey pns
Parts:
- R905, R909, R910: Digi-Key PN 311-5.10KLRCT-ND -> YAG3503CT-ND
Changed lines of the file:
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@@
 			)
 		)
-		(property "Digi-Key PN" "311-5.10KLRCT-ND"
+		(property "Digi-Key PN" "YAG3503CT-ND"
 			(at 195.58 114.3 0)
 			(hide yes)
@@
 			)
 		)
-		(property "Digi-Key PN" "311-5.10KLRCT-ND"
+		(property "Digi-Key PN" "YAG3503CT-ND"
 			(at 208.28 114.3 0)
 			(hide yes)
@@
 			)
 		)
-		(property "Digi-Key PN" "311-5.10KLRCT-ND"
+		(property "Digi-Key PN" "YAG3503CT-ND"
 			(at 111.76 166.37 0)
 			(hide yes)
