File: hdw/DSP_board/rev_a/Audio_Visualiser_DSP/pn_assign_backup_20261008_194741/speaker_signal_conditoning.kicad_sch (KiCad schematic)
At the start: 30 parts, among them J1401 Left, J1402 Right, J1403 Speaker Left TP, J1404 Speaker Right TP, U1401 MCP6N11-001, U1402 MCP6N11-001

Commit message: fix a lot of digikey pns which are out of stock, find alternate inductors, change I2C buffers
Parts:
- U1401, U1402: footprint Package_DFN_QFN:DFN-8-1EP_3x2mm_P0.5mm_EP1.36x1.46mm -> Housings_DFN_QFN:DFN-8-1EP_2x3mm_Pitch0.5mm
Changed lines of the file:
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@@
 			)
 		)
-		(property "Datasheet" "https://services.taiwansemi.com/storage/resources/datasheet/BAT42WS%20SERIES_J2606.pdf"
+		(property "Datasheet" "https://assets.nexperia.com/documents/data-sheet/BAT54J.pdf"
 			(at 134.62 67.31 0)
 			(hide yes)
@@
 			)
 		)
-		(property "Description" "30V 200mA Schottky diode, SOD-323F (TSC BAT43WS)"
+		(property "Description" "30V 200mA Schottky diode, SOD-323F"
 			(at 134.62 67.31 0)
 			(hide yes)
@@
 			)
 		)
-		(property "Sim.Library" "C:\\Users\\drewm\\Documents\\KiCad Projects\\Projects\\audio_visualiser\\hdw\\DSP_board\\rev_a\\sim\\spice_models\\BAT43WS.lib"
+		(property "Sim.Library" "C:\\Users\\drewm\\Documents\\KiCad Projects\\Projects\\audio_visualiser\\hdw\\DSP_board\\rev_a\\sim\\spice_models\\BAT54SW.lib"
 			(at 134.62 67.31 0)
 			(hide yes)
@@
 			)
 		)
-		(property "Sim.Name" "BAT43WS_SOD323F"
+		(property "Sim.Name" "BAT54SW"
 			(at 134.62 67.31 0)
 			(hide yes)
@@
 			)
 		)
-		(property "Sim.Pins" "1=K 2=A"
+		(property "Sim.Pins" "1=2 2=1"
 			(at 134.62 67.31 0)
 			(hide yes)
@@
 			)
 		)
-		(property "Datasheet" "https://services.taiwansemi.com/storage/resources/datasheet/BAT42WS%20SERIES_J2606.pdf"
+		(property "Datasheet" "https://assets.nexperia.com/documents/data-sheet/BAT54J.pdf"
 			(at 116.84 52.07 0)
 			(hide yes)
@@
 			)
 		)
-		(property "Description" "30V 200mA Schottky diode, SOD-323F (TSC BAT43WS)"
+		(property "Description" "30V 200mA Schottky diode, SOD-323F"
 			(at 116.84 52.07 0)
 			(hide yes)
@@
 			)
 		)
-		(property "Sim.Library" "C:\\Users\\drewm\\Documents\\KiCad Projects\\Projects\\audio_visualiser\\hdw\\DSP_board\\rev_a\\sim\\spice_models\\BAT43WS.lib"
+		(property "Sim.Library" "C:\\Users\\drewm\\Documents\\KiCad Projects\\Projects\\audio_visualiser\\hdw\\DSP_board\\rev_a\\sim\\spice_models\\BAT54SW.lib"
 			(at 116.84 52.07 0)
 			(hide yes)
@@
 			)
 		)
-		(property "Sim.Name" "BAT43WS_SOD323F"
+		(property "Sim.Name" "BAT54SW"
 			(at 116.84 52.07 0)
 			(hide yes)
@@
 			)
 		)
-		(property "Sim.Pins" "1=K 2=A"
+		(property "Sim.Pins" "1=2 2=1"
 			(at 116.84 52.07 0)
 			(hide yes)
@@
 			)
 		)
-		(property "Datasheet" "https://services.taiwansemi.com/storage/resources/datasheet/BAT42WS%20SERIES_J2606.pdf"
+		(property "Datasheet" "https://assets.nexperia.com/documents/data-sheet/BAT54J.pdf"
 			(at 134.62 52.07 0)
 			(hide yes)
@@
 			)
 		)
-		(property "Description" "30V 200mA Schottky diode, SOD-323F (TSC BAT43WS)"
+		(property "Description" "30V 200mA Schottky diode, SOD-323F"
 			(at 134.62 52.07 0)
 			(hide yes)
@@
 			)
 		)
-		(property "Sim.Library" "C:\\Users\\drewm\\Documents\\KiCad Projects\\Projects\\audio_visualiser\\hdw\\DSP_board\\rev_a\\sim\\spice_models\\BAT43WS.lib"
+		(property "Sim.Library" "C:\\Users\\drewm\\Documents\\KiCad Projects\\Projects\\audio_visualiser\\hdw\\DSP_board\\rev_a\\sim\\spice_models\\BAT54SW.lib"
 			(at 134.62 52.07 0)
 			(hide yes)
@@
 			)
 		)
-		(property "Sim.Name" "BAT43WS_SOD323F"
+		(property "Sim.Name" "BAT54SW"
 			(at 134.62 52.07 0)
 			(hide yes)
@@
 			)
 		)
-		(property "Sim.Pins" "1=K 2=A"
+		(property "Sim.Pins" "1=2 2=1"
 			(at 134.62 52.07 0)
 			(hide yes)
@@
 			)
 		)
-		(property "Datasheet" "https://services.taiwansemi.com/storage/resources/datasheet/BAT42WS%20SERIES_J2606.pdf"
+		(property "Datasheet" "https://assets.nexperia.com/documents/data-sheet/BAT54J.pdf"
 			(at 116.84 67.31 0)
 			(hide yes)
@@
 			)
 		)
-		(property "Description" "30V 200mA Schottky diode, SOD-323F (TSC BAT43WS)"
+		(property "Description" "30V 200mA Schottky diode, SOD-323F"
 			(at 116.84 67.31 0)
 			(hide yes)
@@
 			)
 		)
-		(property "Sim.Library" "C:\\Users\\drewm\\Documents\\KiCad Projects\\Projects\\audio_visualiser\\hdw\\DSP_board\\rev_a\\sim\\spice_models\\BAT43WS.lib"
+		(property "Sim.Library" "C:\\Users\\drewm\\Documents\\KiCad Projects\\Projects\\audio_visualiser\\hdw\\DSP_board\\rev_a\\sim\\spice_models\\BAT54SW.lib"
 			(at 116.84 67.31 0)
 			(hide yes)
@@
 			)
 		)
-		(property "Sim.Name" "BAT43WS_SOD323F"
+		(property "Sim.Name" "BAT54SW"
 			(at 116.84 67.31 0)
 			(hide yes)
@@
 			)
 		)
-		(property "Sim.Pins" "1=K 2=A"
+		(property "Sim.Pins" "1=2 2=1"
 			(at 116.84 67.31 0)
 			(hide yes)
@@
 			)
 		)
-		(property "Datasheet" "https://services.taiwansemi.com/storage/resources/datasheet/BAT42WS%20SERIES_J2606.pdf"
+		(property "Datasheet" "https://assets.nexperia.com/documents/data-sheet/BAT54J.pdf"
 			(at 116.84 143.51 0)
 			(hide yes)
@@
 			)
 		)
-		(property "Description" "30V 200mA Schottky diode, SOD-323F (TSC BAT43WS)"
+		(property "Description" "30V 200mA Schottky diode, SOD-323F"
 			(at 116.84 143.51 0)
 			(hide yes)
@@
 			)
 		)
-		(property "Sim.Library" "C:\\Users\\drewm\\Documents\\KiCad Projects\\Projects\\audio_visualiser\\hdw\\DSP_board\\rev_a\\sim\\spice_models\\BAT43WS.lib"
+		(property "Sim.Library" "C:\\Users\\drewm\\Documents\\KiCad Projects\\Projects\\audio_visualiser\\hdw\\DSP_board\\rev_a\\sim\\spice_models\\BAT54SW.lib"
 			(at 116.84 143.51 0)
 			(hide yes)
@@
 			)
 		)
-		(property "Sim.Name" "BAT43WS_SOD323F"
+		(property "Sim.Name" "BAT54SW"
 			(at 116.84 143.51 0)
 			(hide yes)
@@
 			)
 		)
-		(property "Sim.Pins" "1=K 2=A"
+		(property "Sim.Pins" "1=2 2=1"
 			(at 116.84 143.51 0)
 			(hide yes)
@@
 			)
 		)
-		(property "Footprint" "Package_DFN_QFN:DFN-8-1EP_3x2mm_P0.5mm_EP1.36x1.46mm"
+		(property "Footprint" "Housings_DFN_QFN:DFN-8-1EP_2x3mm_Pitch0.5mm"
 			(at 160.02 146.05 0)
 			(hide yes)
@@
 			)
 		)
-		(property "Footprint" "Package_DFN_QFN:DFN-8-1EP_3x2mm_P0.5mm_EP1.36x1.46mm"
+		(property "Footprint" "Housings_DFN_QFN:DFN-8-1EP_2x3mm_Pitch0.5mm"
 			(at 160.02 69.85 0)
 			(hide yes)
@@
 			)
 		)
-		(property "Datasheet" "https://services.taiwansemi.com/storage/resources/datasheet/BAT42WS%20SERIES_J2606.pdf"
+		(property "Datasheet" "https://assets.nexperia.com/documents/data-sheet/BAT54J.pdf"
 			(at 116.84 128.27 0)
 			(hide yes)
@@
 			)
 		)
-		(property "Description" "30V 200mA Schottky diode, SOD-323F (TSC BAT43WS)"
+		(property "Description" "30V 200mA Schottky diode, SOD-323F"
 			(at 116.84 128.27 0)
 			(hide yes)
@@
 			)
 		)
-		(property "Sim.Library" "C:\\Users\\drewm\\Documents\\KiCad Projects\\Projects\\audio_visualiser\\hdw\\DSP_board\\rev_a\\sim\\spice_models\\BAT43WS.lib"
+		(property "Sim.Library" "C:\\Users\\drewm\\Documents\\KiCad Projects\\Projects\\audio_visualiser\\hdw\\DSP_board\\rev_a\\sim\\spice_models\\BAT54SW.lib"
 			(at 116.84 128.27 0)
 			(hide yes)
@@
 			)
 		)
-		(property "Sim.Name" "BAT43WS_SOD323F"
+		(property "Sim.Name" "BAT54SW"
 			(at 116.84 128.27 0)
 			(hide yes)
@@
 			)
 		)
-		(property "Sim.Pins" "1=K 2=A"
+		(property "Sim.Pins" "1=2 2=1"
 			(at 116.84 128.27 0)
 			(hide yes)
@@
 			)
 		)
-		(property "Datasheet" "https://services.taiwansemi.com/storage/resources/datasheet/BAT42WS%20SERIES_J2606.pdf"
+		(property "Datasheet" "https://assets.nexperia.com/documents/data-sheet/BAT54J.pdf"
 			(at 134.62 143.51 0)
 			(hide yes)
@@
 			)
 		)
-		(property "Description" "30V 200mA Schottky diode, SOD-323F (TSC BAT43WS)"
+		(property "Description" "30V 200mA Schottky diode, SOD-323F"
 			(at 134.62 143.51 0)
 			(hide yes)
@@
 			)
 		)
-		(property "Sim.Library" "C:\\Users\\drewm\\Documents\\KiCad Projects\\Projects\\audio_visualiser\\hdw\\DSP_board\\rev_a\\sim\\spice_models\\BAT43WS.lib"
+		(property "Sim.Library" "C:\\Users\\drewm\\Documents\\KiCad Projects\\Projects\\audio_visualiser\\hdw\\DSP_board\\rev_a\\sim\\spice_models\\BAT54SW.lib"
 			(at 134.62 143.51 0)
 			(hide yes)
@@
 			)
 		)
-		(property "Sim.Name" "BAT43WS_SOD323F"
+		(property "Sim.Name" "BAT54SW"
 			(at 134.62 143.51 0)
 			(hide yes)
@@
 			)
 		)
-		(property "Sim.Pins" "1=K 2=A"
+		(property "Sim.Pins" "1=2 2=1"
 			(at 134.62 143.51 0)
 			(hide yes)
@@
 			)
 		)
-		(property "Datasheet" "https://services.taiwansemi.com/storage/resources/datasheet/BAT42WS%20SERIES_J2606.pdf"
+		(property "Datasheet" "https://assets.nexperia.com/documents/data-sheet/BAT54J.pdf"
 			(at 134.62 128.27 0)
 			(hide yes)
@@
 			)
 		)
-		(property "Description" "30V 200mA Schottky diode, SOD-323F (TSC BAT43WS)"
+		(property "Description" "30V 200mA Schottky diode, SOD-323F"
 			(at 134.62 128.27 0)
 			(hide yes)
@@
 			)
 		)
-		(property "Sim.Library" "C:\\Users\\drewm\\Documents\\KiCad Projects\\Projects\\audio_visualiser\\hdw\\DSP_board\\rev_a\\sim\\spice_models\\BAT43WS.lib"
+		(property "Sim.Library" "C:\\Users\\drewm\\Documents\\KiCad Projects\\Projects\\audio_visualiser\\hdw\\DSP_board\\rev_a\\sim\\spice_models\\BAT54SW.lib"
 			(at 134.62 128.27 0)
 			(hide yes)
@@
 			)
 		)
-		(property "Sim.Name" "BAT43WS_SOD323F"
+		(property "Sim.Name" "BAT54SW"
 			(at 134.62 128.27 0)
 			(hide yes)
@@
 			)
 		)
-		(property "Sim.Pins" "1=K 2=A"
+		(property "Sim.Pins" "1=2 2=1"
 			(at 134.62 128.27 0)
 			(hide yes)
