File: hdw/DSP_board/rev_a/Audio_Visualiser_DSP/pn_assign_backup_20261008_195349_fp/speaker_signal_conditoning.kicad_sch (KiCad schematic)
At the start: 30 parts, among them J1401 Left, J1402 Right, J1403 Speaker Left TP, J1404 Speaker Right TP, U1401 MCP6N11-001, U1402 MCP6N11-001

Commit message: fix a lot of digikey pns which are out of stock, find alternate inductors, change I2C buffers
Parts:
- U1401, U1402: footprint Package_DFN_QFN:DFN-8-1EP_3x2mm_P0.5mm_EP1.36x1.46mm -> Housings_DFN_QFN:DFN-8-1EP_2x3mm_Pitch0.5mm
Changed lines of the file:
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@@
 			)
 		)
-		(property "Footprint" "Package_DFN_QFN:DFN-8-1EP_3x2mm_P0.5mm_EP1.36x1.46mm"
+		(property "Footprint" "Housings_DFN_QFN:DFN-8-1EP_2x3mm_Pitch0.5mm"
 			(at 160.02 146.05 0)
 			(hide yes)
@@
 			)
 		)
-		(property "Footprint" "Package_DFN_QFN:DFN-8-1EP_3x2mm_P0.5mm_EP1.36x1.46mm"
+		(property "Footprint" "Housings_DFN_QFN:DFN-8-1EP_2x3mm_Pitch0.5mm"
 			(at 160.02 69.85 0)
 			(hide yes)
