File: hdw/DSP_board/rev_a/Audio_Visualiser_DSP/pn_assign_backup_20261008_201544/led_panel_connectors.kicad_sch (KiCad schematic)
At the start: 8 parts, among them J2101 Left, J2102 Right

Commit message: fix a lot of digikey pns which are out of stock, find alternate inductors, change I2C buffers
Parts:
- D2101, D2102, D2103, D2104: value PESD5V0L5UYF -> PESD3V3L5UY; Digi-Key PN 1727-PESD5V0L5UYFCT-ND -> 1727-3828-1-ND
Changed lines of the file:
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@@
 			)
 		)
-		(property "Value" "PESD5V0L5UYF"
+		(property "Value" "PESD3V3L5UY"
 			(at 58.42 66.04 0)
 			(hide yes)
@@
 			)
 		)
-		(property "Digi-Key PN" "1727-PESD5V0L5UYFCT-ND"
+		(property "Digi-Key PN" "1727-3828-1-ND"
 			(at 60.96 66.04 0)
 			(hide yes)
@@
 			)
 		)
-		(property "Value" "PESD5V0L5UYF"
+		(property "Value" "PESD3V3L5UY"
 			(at 87.63 66.04 90)
 			(show_name no)
@@
 			)
 		)
-		(property "Digi-Key PN" "1727-PESD5V0L5UYFCT-ND"
+		(property "Digi-Key PN" "1727-3828-1-ND"
 			(at 99.06 66.04 0)
 			(hide yes)
@@
 			)
 		)
-		(property "Value" "PESD5V0L5UYF"
+		(property "Value" "PESD3V3L5UY"
 			(at 39.37 129.54 0)
 			(hide yes)
@@
 			)
 		)
-		(property "Digi-Key PN" "1727-PESD5V0L5UYFCT-ND"
+		(property "Digi-Key PN" "1727-3828-1-ND"
 			(at 41.91 129.54 0)
 			(hide yes)
@@
 			)
 		)
-		(property "Value" "PESD5V0L5UYF"
+		(property "Value" "PESD3V3L5UY"
 			(at 39.37 66.04 0)
 			(hide yes)
@@
 			)
 		)
-		(property "Digi-Key PN" "1727-PESD5V0L5UYFCT-ND"
+		(property "Digi-Key PN" "1727-3828-1-ND"
 			(at 41.91 66.04 0)
 			(hide yes)
@@
 			)
 		)
-		(property "Value" "PESD5V0L5UYF"
+		(property "Value" "PESD3V3L5UY"
 			(at 64.77 66.04 0)
 			(hide yes)
@@
 			)
 		)
-		(property "Digi-Key PN" "1727-PESD5V0L5UYFCT-ND"
+		(property "Digi-Key PN" "1727-3828-1-ND"
 			(at 67.31 66.04 0)
 			(hide yes)
@@
 			)
 		)
-		(property "Value" "PESD5V0L5UYF"
+		(property "Value" "PESD3V3L5UY"
 			(at 64.77 129.54 0)
 			(hide yes)
@@
 			)
 		)
-		(property "Digi-Key PN" "1727-PESD5V0L5UYFCT-ND"
+		(property "Digi-Key PN" "1727-3828-1-ND"
 			(at 67.31 129.54 0)
 			(hide yes)
@@
 			)
 		)
-		(property "Value" "PESD5V0L5UYF"
+		(property "Value" "PESD3V3L5UY"
 			(at 115.57 129.54 0)
 			(hide yes)
@@
 			)
 		)
-		(property "Digi-Key PN" "1727-PESD5V0L5UYFCT-ND"
+		(property "Digi-Key PN" "1727-3828-1-ND"
 			(at 118.11 129.54 0)
 			(hide yes)
@@
 			)
 		)
-		(property "Value" "PESD5V0L5UYF"
+		(property "Value" "PESD3V3L5UY"
 			(at 52.07 66.04 0)
 			(hide yes)
@@
 			)
 		)
-		(property "Digi-Key PN" "1727-PESD5V0L5UYFCT-ND"
+		(property "Digi-Key PN" "1727-3828-1-ND"
 			(at 54.61 66.04 0)
 			(hide yes)
@@
 			)
 		)
-		(property "Value" "PESD5V0L5UYF"
+		(property "Value" "PESD3V3L5UY"
 			(at 109.22 129.54 0)
 			(hide yes)
@@
 			)
 		)
-		(property "Digi-Key PN" "1727-PESD5V0L5UYFCT-ND"
+		(property "Digi-Key PN" "1727-3828-1-ND"
 			(at 111.76 129.54 0)
 			(hide yes)
@@
 			)
 		)
-		(property "Value" "PESD5V0L5UYF"
+		(property "Value" "PESD3V3L5UY"
 			(at 58.42 129.54 0)
 			(hide yes)
@@
 			)
 		)
-		(property "Digi-Key PN" "1727-PESD5V0L5UYFCT-ND"
+		(property "Digi-Key PN" "1727-3828-1-ND"
 			(at 60.96 129.54 0)
 			(hide yes)
@@
 			)
 		)
-		(property "Value" "PESD5V0L5UYF"
+		(property "Value" "PESD3V3L5UY"
 			(at 115.57 66.04 0)
 			(hide yes)
@@
 			)
 		)
-		(property "Digi-Key PN" "1727-PESD5V0L5UYFCT-ND"
+		(property "Digi-Key PN" "1727-3828-1-ND"
 			(at 118.11 66.04 0)
 			(hide yes)
@@
 			)
 		)
-		(property "Value" "PESD5V0L5UYF"
+		(property "Value" "PESD3V3L5UY"
 			(at 90.17 66.04 0)
 			(hide yes)
@@
 			)
 		)
-		(property "Digi-Key PN" "1727-PESD5V0L5UYFCT-ND"
+		(property "Digi-Key PN" "1727-3828-1-ND"
 			(at 92.71 66.04 0)
 			(hide yes)
@@
 			)
 		)
-		(property "Value" "PESD5V0L5UYF"
+		(property "Value" "PESD3V3L5UY"
 			(at 102.87 66.04 0)
 			(hide yes)
@@
 			)
 		)
-		(property "Digi-Key PN" "1727-PESD5V0L5UYFCT-ND"
+		(property "Digi-Key PN" "1727-3828-1-ND"
 			(at 105.41 66.04 0)
 			(hide yes)
@@
 			)
 		)
-		(property "Value" "PESD5V0L5UYF"
+		(property "Value" "PESD3V3L5UY"
 			(at 102.87 129.54 0)
 			(hide yes)
@@
 			)
 		)
-		(property "Digi-Key PN" "1727-PESD5V0L5UYFCT-ND"
+		(property "Digi-Key PN" "1727-3828-1-ND"
 			(at 105.41 129.54 0)
 			(hide yes)
@@
 			)
 		)
-		(property "Value" "PESD5V0L5UYF"
+		(property "Value" "PESD3V3L5UY"
 			(at 36.83 129.54 90)
 			(show_name no)
@@
 			)
 		)
-		(property "Digi-Key PN" "1727-PESD5V0L5UYFCT-ND"
+		(property "Digi-Key PN" "1727-3828-1-ND"
 			(at 48.26 129.54 0)
 			(hide yes)
@@
 			)
 		)
-		(property "Value" "PESD5V0L5UYF"
+		(property "Value" "PESD3V3L5UY"
 			(at 109.22 66.04 0)
 			(hide yes)
@@
 			)
 		)
-		(property "Digi-Key PN" "1727-PESD5V0L5UYFCT-ND"
+		(property "Digi-Key PN" "1727-3828-1-ND"
 			(at 111.76 66.04 0)
 			(hide yes)
@@
 			)
 		)
-		(property "Value" "PESD5V0L5UYF"
+		(property "Value" "PESD3V3L5UY"
 			(at 90.17 129.54 0)
 			(hide yes)
@@
 			)
 		)
-		(property "Digi-Key PN" "1727-PESD5V0L5UYFCT-ND"
+		(property "Digi-Key PN" "1727-3828-1-ND"
 			(at 92.71 129.54 0)
 			(hide yes)
@@
 			)
 		)
-		(property "Value" "PESD5V0L5UYF"
+		(property "Value" "PESD3V3L5UY"
 			(at 36.83 66.04 90)
 			(show_name no)
@@
 			)
 		)
-		(property "Digi-Key PN" "1727-PESD5V0L5UYFCT-ND"
+		(property "Digi-Key PN" "1727-3828-1-ND"
 			(at 48.26 66.04 0)
 			(hide yes)
@@
 			)
 		)
-		(property "Value" "PESD5V0L5UYF"
+		(property "Value" "PESD3V3L5UY"
 			(at 87.63 129.54 90)
 			(show_name no)
@@
 			)
 		)
-		(property "Digi-Key PN" "1727-PESD5V0L5UYFCT-ND"
+		(property "Digi-Key PN" "1727-3828-1-ND"
 			(at 99.06 129.54 0)
 			(hide yes)
@@
 			)
 		)
-		(property "Value" "PESD5V0L5UYF"
+		(property "Value" "PESD3V3L5UY"
 			(at 52.07 129.54 0)
 			(hide yes)
@@
 			)
 		)
-		(property "Digi-Key PN" "1727-PESD5V0L5UYFCT-ND"
+		(property "Digi-Key PN" "1727-3828-1-ND"
 			(at 54.61 129.54 0)
 			(hide yes)
