File: hdw/DSP_board/rev_a/Audio_Visualiser_DSP/pn_assign_backup_20261008_202005/dspic33_gpio.kicad_sch (KiCad schematic)
At the start: 20 parts, among them J801 Boot Audio Source Select, U801 PCA9536DP, U802 74LVC1G97, U803 TCA9801, U804 dsPIC33AK256MPS105, U805 74LVC1G97

Commit message: fix a lot of digikey pns which are out of stock, find alternate inductors, change I2C buffers
Parts:
- U803: value TCA9801 -> TCA9803; Digi-Key PN 296-47828-1-ND -> 296-47829-1-ND
Changed lines of the file:
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@@
 			)
 		)
-		(property "Value" "TCA9801"
+		(property "Value" "TCA9803"
 			(at 138.43 132.08 0)
 			(show_name no)
@@
 			)
 		)
-		(property "Digi-Key PN" "296-47828-1-ND"
+		(property "Digi-Key PN" "296-47829-1-ND"
 			(at 133.35 143.51 0)
 			(hide yes)
