File: hdw/DSP_board/rev_a/Audio_Visualiser_DSP/pn_assign_backup_20261008_202005/led_panel_buffers.kicad_sch (KiCad schematic)
At the start: 29 parts, among them U1801 74LVC1G97, U1802 74LVC1G97, U1803 74VHC541BQ,115, U1804 74VHC541BQ,115, U1805 74LVC1G97, U1806 74LVC1G97, U1807 TCA9801, U1808 74LVC1G97, U1809 TCA9801

Commit message: fix a lot of digikey pns which are out of stock, find alternate inductors, change I2C buffers
Parts:
- U1807, U1809: value TCA9801 -> TCA9803; Digi-Key PN 296-47828-1-ND -> 296-47829-1-ND
Changed lines of the file:
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@@
 			)
 		)
-		(property "Value" "TCA9801"
+		(property "Value" "TCA9803"
 			(at 217.17 25.4 0)
 			(show_name no)
@@
 			)
 		)
-		(property "Digi-Key PN" "296-47828-1-ND"
+		(property "Digi-Key PN" "296-47829-1-ND"
 			(at 212.09 36.83 0)
 			(hide yes)
@@
 			)
 		)
-		(property "Value" "TCA9801"
+		(property "Value" "TCA9803"
 			(at 217.17 114.3 0)
 			(show_name no)
@@
 			)
 		)
-		(property "Digi-Key PN" "296-47828-1-ND"
+		(property "Digi-Key PN" "296-47829-1-ND"
 			(at 212.09 125.73 0)
 			(hide yes)
